File: hardware/schematics/kicad/front_panel.kicad_sch (KiCad schematic)
At the start: 0 parts

Commit message: splitting schematic into blocks
Parts:
- added DIS1, DIS2: ~, led-displays-obsolete:TIL311, symbol main-eagle-import:HTIL311A
- added IC113: 7404N, Package_DIP:DIP-14_W7.62mm, symbol main-eagle-import:7404N
- added IC114: 74377N, Package_DIP:DIP-20_W7.62mm, symbol main-eagle-import:74377N
- added IC115, IC185: 74244N, Package_DIP:DIP-20_W7.62mm, symbol main-eagle-import:74244N
- added IC155, IC156: 74257N, Package_DIP:DIP-16_W7.62mm, symbol main-eagle-import:74257N
- added IC164, IC170: 7474N, Package_DIP:DIP-14_W7.62mm, symbol main-eagle-import:7474N
- added IC175, IC187: 74279N, Package_DIP:DIP-16_W7.62mm, symbol main-eagle-import:74279N
- added IC186, IC198, IC200, IC202, IC203, IC204: 74244N, Package_DIP:DIP-20_W7.62mm, symbol main-eagle-import:74xx-eu_74244N
- added RN1, RN3, RN4, RN5, RN6, RN7, RN8: R_Pack08, Package_DIP:DIP-16_W7.62mm, symbol Device:R_Pack08
- added S1: 100SP1T1B4M2QE, kicad_models:SW_100SP1T1B4M2QE, symbol SPDT_Switch:100SP1T1B4M2QE
- added SW1, SW11, SW2, SW5: SW_SPST, kicad_models:SW_100SP1T1B4M2QE, symbol Switch:SW_SPST
- added SW10, SW12, SW3, SW4, SW6, SW7, SW8, SW9: SW_DIP_x08, Package_DIP:DIP-16_W7.62mm, symbol Switch:SW_DIP_x08
- added U16: 4040, Package_DIP:DIP-16_W7.62mm, symbol 4xxx:4040
- added U18: 74HC04, Package_DIP:DIP-14_W7.62mm, symbol 74xx:74HC04
- added U23: 74LS173, Package_DIP:DIP-16_W7.62mm, symbol 74xx:74LS173
- added X1: ACO-10MHz, Oscillator:Oscillator_DIP-14, symbol Oscillator:ACO-xxxMHz
Connections:
- new net: U18.5, U23.3 (Q0)
- new net: SW3.10, SW3.11, SW3.12, SW3.13, SW3.14, SW3.15, SW3.16, SW3.9, U18.3, U23.7 (Cp)
- new net: RN5.7 (R7.1), SW8.2
- new net: RN5.8 (R8.1), SW8.1
- new net: IC185.2 (A1), SW12.10, SW12.11, SW12.12, SW12.13, SW12.14, SW12.15, SW12.16, SW12.9
- new net: IC115.5 (Y3), IC156.10 (3B)
- new net: IC114.16 (7Q), IC156.11 (3A)
- new net: IC115.3 (Y4), IC156.13 (4B)
- new net: IC114.19 (8Q), IC156.14 (4A)
- new net: IC155.15 (G), IC156.15 (G)
- new net: IC114.12 (5Q), IC156.2 (1A)
- new net: IC115.9 (Y1), IC156.3 (1B)
- new net: IC114.15 (6Q), IC156.5 (2A)
- new net: IC115.7 (Y2), IC156.6 (2B)
- new net: IC187.5 (R), RN7.1 (R1.1), SW10.8
- new net: IC187.6 (S), RN7.2 (R2.1), SW10.7
- new net: IC170.3 (CLK), U18.4
- new net: IC164.2 (D), RN8.8 (R8.1), SW11.2 (B)
- new net: IC164.12 (D), RN8.1 (R1.1), SW2.2 (B)
- new net: IC187.10 (R), RN7.3 (R3.1), SW10.6
- new net: IC187.11 (S1), IC187.12 (S2), RN7.4 (R4.1), SW10.5
- new net: IC187.1 (R), RN7.5 (R5.1), SW10.4
- new net: IC187.2 (S1), IC187.3 (S2), RN7.6 (R6.1), SW10.3
- new net: RN1.1 (R1.1), SW4.8
- new net: RN1.2 (R2.1), SW4.7
- new net: RN1.3 (R3.1), SW4.6
- new net: IC113.4 (O), IC114.1 (G)
- new net: IC115.14 (Y3), IC155.10 (3B)
- new net: IC114.6 (3Q), IC155.11 (3A)
- new net: IC115.12 (Y4), IC155.13 (4B)
- new net: IC114.9 (4Q), IC155.14 (4A)
- new net: IC114.2 (1Q), IC155.2 (1A)
- new net: IC115.18 (Y1), IC155.3 (1B)
- new net: IC114.5 (2Q), IC155.5 (2A)
- new net: IC115.16 (Y2), IC155.6 (2B)
- new net: SW3.8, U16.13 (Q7)
- new net: SW3.6, U16.2 (Q5)
- new net: SW3.5, U16.3 (Q4)
- new net: SW3.7, U16.4 (Q6)
- new net: SW3.4, U16.5 (Q3)
- new net: SW3.3, U16.6 (Q2)
- new net: SW3.2, U16.7 (Q1)
- new net: SW3.1, U16.9 (Q0)
- new net GND: DIS1.10 (DP-R), DIS1.4 (DP-L), DIS1.5 (L-SI), DIS1.7 (GND), DIS1.8 (BI), DIS2.10 (DP-R), DIS2.4 (DP-L), DIS2.5 (L-SI), DIS2.7 (GND), DIS2.8 (BI), IC115.1 (G), IC115.19 (G), IC185.1 (G), IC185.4 (A2), IC185.6 (A3), IC185.8 (A4), IC186.1 (G), IC186.8 (A4), IC198.1 (G), IC198.19 (G), IC200.1 (G), IC200.19 (G), IC202.1 (G), IC202.15 (A3), IC202.17 (A4), IC202.19 (G), IC203.1 (G), IC203.19 (G), IC203.2 (A1), IC203.4 (A2), IC203.6 (A3), IC203.8 (A4), IC204.1 (G), RN8.10 (R7.2), RN8.11 (R6.2), RN8.12 (R5.2), RN8.13 (R4.2), RN8.14 (R3.2), RN8.15 (R2.2), RN8.16 (R1.2), RN8.9 (R8.2), S1.2, SW10.10, SW10.11, SW10.12, SW10.13, SW10.14, SW10.15, SW10.16, SW10.9, SW4.10, SW4.11, SW4.12, SW4.13, SW4.14, SW4.15, SW4.16, SW4.9, SW6.10, SW6.11, SW6.12, SW6.13, SW6.14, SW6.15, SW6.16, SW6.9, SW7.10, SW7.11, SW7.12, SW7.13, SW7.14, SW7.15, SW7.16, SW7.9, SW8.10, SW8.11, SW8.12, SW8.13, SW8.14, SW8.15, SW8.16, SW8.9, SW9.10, SW9.11, SW9.12, SW9.13, SW9.14, SW9.15, SW9.16, SW9.9, U16.11 (Reset), U16.8 (VSS), U23.1 (Oe1), U23.11 (D3), U23.12 (D2), U23.13 (D1), U23.2 (Oe2), U23.8 (GND), X1.7 (GND)
- new net address_bus0: IC198.18 (Y1)
- new net address_bus1: IC198.16 (Y2)
- new net address_bus10: IC200.14 (Y3)
- new net address_bus11: IC200.12 (Y4)
- new net address_bus12: IC200.9 (Y1)
- new net address_bus13: IC200.7 (Y2)
- new net address_bus14: IC200.5 (Y3)
- new net address_bus15: IC200.3 (Y4)
- new net address_bus16: IC202.18 (Y1)
- new net address_bus17: IC202.16 (Y2)
- new net address_bus18: IC202.14 (Y3)
- new net address_bus19: IC202.12 (Y4)
- new net address_bus2: IC198.14 (Y3)
- new net address_bus20: IC202.9 (Y1)
- new net address_bus21: IC202.7 (Y2)
- new net address_bus3: IC198.12 (Y4)
- new net address_bus4: IC198.9 (Y1)
- new net address_bus5: IC198.7 (Y2)
- new net address_bus6: IC198.5 (Y3)
- new net address_bus7: IC198.3 (Y4)
- new net address_bus8: IC200.18 (Y1)
- new net address_bus9: IC200.16 (Y2)
- new net bus_mem_io: IC186.14 (Y3)
- new net bus_rd: IC186.18 (Y1)
- new net bus_tristate: IC155.1 (~{A}/B), IC156.1 (~{A}/B)
- new net bus_wr: IC186.16 (Y2)
- new net clk: IC114.11 (CLK), IC164.11 (CLK), IC164.3 (CLK), IC185.18 (Y1), U18.9
- new net clk_10mhz: U16.10 (CLK), X1.8 (OUT)
- new net clk_crystal: SW12.2, U18.6, U23.14 (D0)
- new net data_bus0: IC203.9 (Y1)
- new net data_bus1: IC203.7 (Y2)
- new net data_bus2: IC203.5 (Y3)
- new net data_bus3: IC203.3 (Y4)
- new net data_bus4: IC204.18 (Y1)
- new net data_bus5: IC204.16 (Y2)
- new net data_bus6: IC204.14 (Y3)
- new net data_bus7: IC204.12 (Y4)
- new net display_reg_load: IC113.3 (I)
- new net display_register0: DIS1.3 (D0), IC155.4 (1Y)
- new net display_register1: DIS1.2 (D1), IC155.7 (2Y)
- new net display_register2: DIS1.13 (D2), IC155.9 (3Y)
- new net display_register3: DIS1.12 (D3), IC155.12 (4Y)
- new net display_register4: DIS2.3 (D0), IC156.4 (1Y)
- new net display_register5: DIS2.2 (D1), IC156.7 (2Y)
- new net display_register6: DIS2.13 (D2), IC156.9 (3Y)
- new net display_register7: DIS2.12 (D3), IC156.12 (4Y)
- new net dma_req: IC164.5 (Q)
- new net ext_input: IC164.9 (Q)
- new net panel_address_0: IC198.2 (A1), RN4.1 (R1.1), SW7.8
- new net panel_address_1: IC198.4 (A2), RN4.2 (R2.1), SW7.7
- new net panel_address_10: IC200.6 (A3), RN3.3 (R3.1), SW6.6
- new net panel_address_11: IC200.8 (A4), RN3.4 (R4.1), SW6.5
- new net panel_address_12: IC200.11 (A1), RN3.5 (R5.1), SW6.4
- new net panel_address_13: IC200.13 (A2), RN3.6 (R6.1), SW6.3
- new net panel_address_14: IC200.15 (A3), RN3.7 (R7.1), SW6.2
- new net panel_address_15: IC200.17 (A4), RN3.8 (R8.1), SW6.1
- new net panel_address_16: IC202.2 (A1), RN5.1 (R1.1), SW8.8
- new net panel_address_17: IC202.4 (A2), RN5.2 (R2.1), SW8.7
- new net panel_address_18: IC202.6 (A3), RN5.3 (R3.1), SW8.6
- new net panel_address_19: IC202.8 (A4), RN5.4 (R4.1), SW8.5
- new net panel_address_2: IC198.6 (A3), RN4.3 (R3.1), SW7.6
- new net panel_address_20: IC202.11 (A1), RN5.5 (R5.1), SW8.4
- new net panel_address_21: IC202.13 (A2), RN5.6 (R6.1), SW8.3
- new net panel_address_3: IC198.8 (A4), RN4.4 (R4.1), SW7.5
- new net panel_address_4: IC198.11 (A1), RN4.5 (R5.1), SW7.4
- new net panel_address_5: IC198.13 (A2), RN4.6 (R6.1), SW7.3
- new net panel_address_6: IC198.15 (A3), RN4.7 (R7.1), SW7.2
- new net panel_address_7: IC198.17 (A4), RN4.8 (R8.1), SW7.1
- new net panel_address_8: IC200.2 (A1), RN3.1 (R1.1), SW6.8
- new net panel_address_9: IC200.4 (A2), RN3.2 (R2.1), SW6.7
- new net panel_data_0: IC203.11 (A1), RN6.1 (R1.1), SW9.8
- new net panel_data_1: IC203.13 (A2), RN6.2 (R2.1), SW9.7
- new net panel_data_2: IC203.15 (A3), RN6.3 (R3.1), SW9.6
- new net panel_data_3: IC203.17 (A4), RN6.4 (R4.1), SW9.5
- new net panel_data_4: IC204.2 (A1), RN6.5 (R5.1), SW9.4
- new net panel_data_5: IC204.4 (A2), RN6.6 (R6.1), SW9.3
- new net panel_data_6: IC204.6 (A3), RN6.7 (R7.1), SW9.2
- new net panel_data_7: IC204.8 (A4), RN6.8 (R8.1), SW9.1
- new net panel_mem_io: IC186.6 (A3), IC187.4 (Q)
- new net panel_rd: IC186.2 (A1), IC187.9 (Q)
- new net panel_regsel_0: RN1.8 (R8.1), SW4.1
- new net panel_regsel_1: RN1.7 (R7.1), SW4.2
- new net panel_regsel_2: RN1.6 (R6.1), SW4.3
- new net panel_regsel_3: RN1.5 (R5.1), SW4.4
- new net panel_regsel_4: RN1.4 (R4.1), SW4.5
- new net panel_wr: IC186.4 (A2), IC187.7 (Q)
- new net reset: IC175.1 (R), S1.3
- new net rst: RN8.2 (R2.1), SW1.2 (B), U18.1, U23.15 (Mr)
- new net set: IC175.2 (S1), IC175.3 (S2), S1.1
- new net single_step_clk: IC175.4 (Q), SW12.1
- new net stop_clk_req: IC170.2 (D), RN8.7 (R7.1), SW5.2 (B)
- new net stop_clock: IC170.5 (Q), U23.10 (E2), U23.9 (E1)
- new net vcc: DIS1.14 (VCC), DIS2.14 (VCC), IC164.1 (CLR), IC164.10 (PRE), IC164.13 (CLR), IC164.4 (PRE), IC170.1 (CLR), IC170.4 (PRE), RN1.10 (R7.2), RN1.11 (R6.2), RN1.12 (R5.2), RN1.13 (R4.2), RN1.14 (R3.2), RN1.15 (R2.2), RN1.16 (R1.2), RN1.9 (R8.2), RN3.10 (R7.2), RN3.11 (R6.2), RN3.12 (R5.2), RN3.13 (R4.2), RN3.14 (R3.2), RN3.15 (R2.2), RN3.16 (R1.2), RN3.9 (R8.2), RN4.10 (R7.2), RN4.11 (R6.2), RN4.12 (R5.2), RN4.13 (R4.2), RN4.14 (R3.2), RN4.15 (R2.2), RN4.16 (R1.2), RN4.9 (R8.2), RN5.10 (R7.2), RN5.11 (R6.2), RN5.12 (R5.2), RN5.13 (R4.2), RN5.14 (R3.2), RN5.15 (R2.2), RN5.16 (R1.2), RN5.9 (R8.2), RN6.10 (R7.2), RN6.11 (R6.2), RN6.12 (R5.2), RN6.13 (R4.2), RN6.14 (R3.2), RN6.15 (R2.2), RN6.16 (R1.2), RN6.9 (R8.2), RN7.11 (R6.2), RN7.12 (R5.2), RN7.13 (R4.2), RN7.14 (R3.2), RN7.15 (R2.2), RN7.16 (R1.2), SW1.1 (A), SW11.1 (A), SW2.1 (A), SW5.1 (A), U16.16 (VDD), U23.16 (VCC), X1.14 (Vcc)
- new net w0: IC114.3 (1D), IC115.2 (A1)
- new net w1: IC114.4 (2D), IC115.4 (A2)
- new net w2: IC114.7 (3D), IC115.6 (A3)
- new net w3: IC114.8 (4D), IC115.8 (A4)
- new net w4: IC114.13 (5D), IC115.11 (A1)
- new net w5: IC114.14 (6D), IC115.13 (A2)
- new net w6: IC114.17 (7D), IC115.15 (A3)
- new net w7: IC114.18 (8D), IC115.17 (A4)
- new net ~{clk}: U18.8
- new net ~{rst}: U18.2
- no-connect marks 0 -> 36
Other:
- note added: "IMPROVE THIS PART OF THE CIRCUIT"
- note added: "front panel register display"
- note added: "should add resistor here at clock select output because if clock floats, it could make stop_clock signal meta stable"
- note added: "single step clock"
