File: hardware/schematics/kicad/main.kicad_sch (KiCad schematic)
At the start: 301 parts, among them IC1 74377N, IC10 74153N, IC100 74273N, IC101 74273N, IC102 74273N, IC103 74273N, IC104 74273N, IC105 74273N, IC106 74273N, IC107 74273N, IC108 74273N, IC109 7427N, IC11 74257N, IC110 74245N, IC111 74257N, IC112 74257N, IC113 7404N, IC114 74377N, IC115 74244N, IC116 74138N, IC117 74244N, IC118 74244N, IC119 74244N, IC12 74257N, IC120 74244N, IC121 7404N, IC122 7420N, IC123 74151N, IC124 74151N, IC125 74151N, IC126 74151N, IC127 74151N, IC128 74151N, IC129 74151N, IC13 7408N, IC130 74151N, IC131 74151N, IC132 74151N, IC133 74151N, IC134 74151N, IC135 74151N, IC136 74151N, IC137 74151N, IC138 74151N, IC139 74151N, IC14 74153N, IC140 74151N, IC141 74151N, IC142 74151N, IC143 74151N, IC144 74151N, IC145 74151N, IC146 74151N, IC147 74151N, IC148 74151N, IC149 74151N, IC15 74257N, IC150 74151N, IC151 74151N, IC152 74151N, IC153 74151N, IC154 74151N, IC155 74257N, IC156 74257N, IC157 74257N, IC158 74257N, IC159 74257N, IC16 74257N, IC160 74257N, IC161 7408N, IC162 7430N, IC163 7404N, IC164 7474N, IC165 7427N, IC166 74153N, IC167 74153N, IC168 74153N, IC169 74153N, IC17 74153N, IC170 7474N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

Commit message: all backdated commits
Parts:
- added unit 2 of ALU_HIGH1
- added unit 2 of ALU_LOW1
Connections:
- net GND: now also ALU_HIGH1.12 (GND), ALU_LOW1.12 (GND)
- net vcc: now also ALU_HIGH1.24 (VCC), ALU_LOW1.24 (VCC)

Commit message: schem cleanup
Other:
- added sheet front_panel (front_panel.kicad_sch)
- added sheet memory_peripherals (memory_peripherals.kicad_sch)
- added sheet microcode_alu (microcode_alu.kicad_sch)
- added sheet registers_paging (registers_paging.kicad_sch)
Changed lines of the file:
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@@
+		)
+	)
+	(sheet
+		(at 86.36 877.57)
+		(size 247.65 151.13)
+		(fields_autoplaced yes)
+		(stroke
+			(width 0.1524)
+			(type solid)
+		)
+		(fill
+			(color 0 0 0 0.0000)
+		)
+		(property "Sheetname" "microcode_alu"
+			(at 86.36 876.8584 0)
+			(show_name yes)
+			(effects
+				(font
+					(size 1.27 1.27)
+				)
+				(justify left bottom)
+			)
+		)
+		(property "Sheetfile" "microcode_alu.kicad_sch"
+			(at 86.36 1029.2846 0)
+			(show_name yes)
+			(effects
+				(font
+					(size 1.27 1.27)
+				)
+				(justify left top)
+			)
+		)
+		(instances
+			(project "main"
+				(path "/8dc530de-176d-4542-9ed1-97157904b8fd"
+					(page "2")
+				)
+			)
+		)
+	)
+	(sheet
+		(at 85.09 1062.99)
+		(size 157.48 114.3)
+		(fields_autoplaced yes)
+		(stroke
+			(width 0.1524)
+			(type solid)
+		)
+		(fill
+			(color 0 0 0 0.0000)
+		)
+		(property "Sheetname" "registers_paging"
+			(at 85.09 1062.2784 0)
+			(show_name yes)
+			(effects
+				(font
+					(size 1.27 1.27)
+				)
+				(justify left bottom)
+			)
+		)
+		(property "Sheetfile" "registers_paging.kicad_sch"
+			(at 85.09 1177.8746 0)
+			(show_name yes)
+			(effects
+				(font
+					(size 1.27 1.27)
+				)
+				(justify left top)
+			)
+		)
+		(instances
+			(project "main"
+				(path "/8dc530de-176d-4542-9ed1-97157904b8fd"
+					(page "3")
+				)
+			)
+		)
+	)
+	(sheet
+		(at 360.68 876.3)
+		(size 179.07 157.48)
+		(fields_autoplaced yes)
+		(stroke
+			(width 0.1524)
+			(type solid)
+		)
+		(fill
+			(color 0 0 0 0.0000)
+		)
+		(property "Sheetname" "memory_peripherals"
+			(at 360.68 875.5884 0)
+			(effects
+				(font
+					(size 1.27 1.27)
+				)
+				(justify left bottom)
+			)
+		)
+		(property "Sheetfile" "memory_peripherals.kicad_sch"
+			(at 360.68 1034.3646 0)
+			(effects
+				(font
+					(size 1.27 1.27)
+				)
+				(justify left top)
+			)
+		)
+		(instances
+			(project "main"
+				(path "/8dc530de-176d-4542-9ed1-97157904b8fd"
+					(page "4")
+				)
+			)
+		)
+	)
+	(sheet
+		(at 294.64 1064.26)
+		(size 146.05 111.76)
+		(fields_autoplaced yes)
+		(stroke
+			(width 0.1524)
+			(type solid)
+		)
+		(fill
+			(color 0 0 0 0.0000)
+		)
+		(property "Sheetname" "front_panel"
+			(at 294.64 1063.5484 0)
+			(effects
+				(font
+					(size 1.27 1.27)
+				)
+				(justify left bottom)
+			)
+		)
+		(property "Sheetfile" "front_panel.kicad_sch"
+			(at 294.64 1176.6046 0)
+			(effects
+				(font
+					(size 1.27 1.27)
+				)
+				(justify left top)
+			)
+		)
+		(instances
+			(project "main"
+				(path "/8dc530de-176d-4542-9ed1-97157904b8fd"
+					(page "5")
+				)
+			)
 		)
 	)

Commit message: splitting schematic into blocks
Parts:
- removed ALU_HIGH1, ALU_LOW1: 74181N, Package_DIP:DIP-24_W7.62mm, symbol main-eagle-import:74181N
- removed BIOS_ROM1, U_ROM1, U_ROM10, U_ROM11, U_ROM12, U_ROM13, U_ROM14, U_ROM15, U_ROM2, U_ROM3, U_ROM4, U_ROM5, U_ROM6, U_ROM7, U_ROM8, U_ROM9: 27512, Package_DIP:DIP-28_W15.24mm, symbol main-eagle-import:27512
- removed C1: C, Capacitor_THT:C_Disc_D7.5mm_W4.4mm_P5.00mm, symbol Device:C
- removed DIS1, DIS2: ~, led-displays-obsolete:TIL311, symbol main-eagle-import:HTIL311A
- removed FLAGS1, IC100, IC101, IC102, IC103, IC104, IC105, IC106, IC107, IC108, IC22, IC91, IC92, IC94, IC95, IC96, IC97, IC98, IC99, IRQ_STATUS_1: 74273N, Package_DIP:DIP-20_W7.62mm, symbol main-eagle-import:74273N
- removed IC1, IC114, IC195, IC2, IC36, IC42, IC54, IC55, IC56, IC57, IC58, IC59, IC60, IC61, IC62, IC63, IC64, IC65, IC66, IC67, IC68, IC69, IC70, IC71, IC72, IC73, IC74, IC84, IC85, IRQ_CODE1, MARH1, MARL1, MDRH1, MDRL1: 74377N, Package_DIP:DIP-20_W7.62mm, symbol main-eagle-import:74377N
- removed IC10, IC14, IC166, IC167, IC168, IC169, IC17, IC18, IC7, IC77, IC78, IC79, IC8, IC80, IC81, IC82, IC83, IC87, IC89, IC9: 74153N, Package_DIP:DIP-16_W7.62mm, symbol main-eagle-import:74153N
- removed IC109, IC165, IC51: 7427N, Package_DIP:DIP-14_W7.62mm, symbol main-eagle-import:7427N
- removed IC11, IC111, IC112, IC12, IC15, IC155, IC156, IC157, IC158, IC159, IC16, IC160, IC19, IC190, IC191, IC20, IC24, IC25, IC26, IC27, IC30, IC76, IC93: 74257N, Package_DIP:DIP-16_W7.62mm, symbol main-eagle-import:74257N
- removed IC110: 74245N, Package_DIP:DIP-20_W7.62mm, symbol main-eagle-import:74245N
- removed IC113, IC121, IC163, IC194, IC21, IC43: 7404N, Package_DIP:DIP-14_W7.62mm, symbol main-eagle-import:7404N
- removed IC115, IC117, IC118, IC119, IC120, IC172, IC173, IC174, IC179, IC180, IC185, IC197: 74244N, Package_DIP:DIP-20_W7.62mm, symbol main-eagle-import:74244N
- removed IC116, IC176, IC199, IC86, IRQ_RST_DECODER1: 74138N, Package_DIP:DIP-16_W7.62mm, symbol main-eagle-import:74138N
- removed IC122: 7420N, Package_DIP:DIP-14_W7.62mm, symbol main-eagle-import:7420N
- removed IC123, IC124, IC125, IC126, IC127, IC128, IC129, IC130, IC131, IC132, IC133, IC134, IC135, IC136, IC137, IC138, IC139, IC140, IC141, IC142, IC143, IC144, IC145, IC146, IC147, IC148, IC149, IC150, IC151, IC152, IC153, IC154, IC28, IC49, IC50, IC88, IC90: 74151N, Package_DIP:DIP-16_W7.62mm, symbol main-eagle-import:74151N
- removed IC13, IC161, IC35, IRQ_AND_1, IRQ_AND_2: 7408N, Package_DIP:DIP-14_W7.62mm, symbol main-eagle-import:7408N
- removed IC162: 7430N, Package_DIP:DIP-14_W7.62mm, symbol main-eagle-import:7430N
- removed IC164, IC170, IRQ_0_DFF1, IRQ_1_DFF1, IRQ_2_DFF1, IRQ_3_DFF1: 7474N, Package_DIP:DIP-14_W7.62mm, symbol main-eagle-import:7474N
- removed IC171, IC188, IC192, IC29, IC44, IC45, IC48, IC53: 7432N, Package_DIP:DIP-14_W7.62mm, symbol main-eagle-import:7432N
- removed IC175, IC187: 74279N, Package_DIP:DIP-16_W7.62mm, symbol main-eagle-import:74279N
- removed IC177, IC178: 58C256P, Package_DIP:DIP-28_W15.24mm, symbol main-eagle-import:58C256P
- removed IC181, IC182, IC183, IC184, MDR_IN_MUX_1, MDR_IN_MUX_2, MDR_OUT_MUX_1, MDR_OUT_MUX_2: 74157N, Package_DIP:DIP-16_W7.62mm, symbol main-eagle-import:74157N
- removed IC186, IC196, IC198, IC200, IC202, IC204, IC206, IC47: 74244N, Package_DIP:DIP-20_W7.62mm, symbol main-eagle-import:74xx-eu_74244N
- removed IC189: ~, main:DIL14, symbol main-eagle-import:7408N
- removed IC193: ~, main:DIL14, symbol main-eagle-import:7432N
- removed IC201: ~, main:DIL14, symbol main-eagle-import:7404N
- removed IC23, IC_10_1, IC_10_2: 7410N, Package_DIP:DIP-14_W7.62mm, symbol main-eagle-import:7410N
- removed IC3, IC31, IC32, IC33, IC34, IC4, IC5, IC6: 74253N, Package_DIP:DIP-16_W7.62mm, symbol main-eagle-import:74253N
- removed IC37, IC_86_1, IC_86_2: 7486N, Package_DIP:DIP-14_W7.62mm, symbol main-eagle-import:7486N
- removed IC38, IC39, IC40, IC41: 74283N, Package_DIP:DIP-16_W7.62mm, symbol main-eagle-import:74283N
- removed IC46, IC52: 7400N, Package_DIP:DIP-14_W7.62mm, symbol main-eagle-import:7400N
- removed IC75: 7411N, Package_DIP:DIP-14_W7.62mm, symbol main-eagle-import:7411N
- removed IC_02_1: 7402N, Package_DIP:DIP-14_W7.62mm, symbol main-eagle-import:7402N
- removed IC_04_1: 7404N, Package_DIP:DIP-14_W7.62mm, symbol main-eagle-import:74xx-eu_7404N
- removed IRQ_ENCODER1: 74148N, Package_DIP:DIP-16_W7.62mm, symbol main-eagle-import:74148N
- removed J1: Conn_02x17_Odd_Even, symbol Connector_Generic:Conn_02x17_Odd_Even
- removed PIO_0: 8255, Package_DIP:DIP-40_W15.24mm, symbol Interface:8255
- removed RN1, RN2, RN3, RN4, RN5, RN6, RN7, RN8, RN9: R_Pack08, Package_DIP:DIP-16_W7.62mm, symbol Device:R_Pack08
- removed S1: 100SP1T1B4M2QE, kicad_models:SW_100SP1T1B4M2QE, symbol SPDT_Switch:100SP1T1B4M2QE
- removed SW1, SW11, SW12, SW13: SW_SPST, kicad_models:SW_100SP1T1B4M2QE, symbol Switch:SW_SPST
- removed SW10, SW2, SW4, SW5, SW6, SW7, SW8, SW9: SW_DIP_x08, Package_DIP:DIP-16_W7.62mm, symbol Switch:SW_DIP_x08
- removed U1, U2, U3, U4, U5, U6, U7, U8: as6c4008-55pcn, Package_DIP:DIP-32_W15.24mm, symbol main-eagle-import:AS6C4008-55PCN
- removed U10: 8253, Package_DIP:DIP-24_W15.24mm, symbol Timer:8253
- removed U11: 74LS06, symbol 74xx:74LS06
- removed U12: 74LS377, symbol 74xx:74LS377
- removed U13, U14: 16550, Package_DIP:DIP-40_W15.24mm, symbol Interface_UART:16550
- removed U15: KM62256CLP, Package_DIP:DIP-28_W15.24mm, symbol Memory_RAM:KM62256CLP
- removed U16: 4040, Package_DIP:DIP-16_W7.62mm, symbol 4xxx:4040
- removed U17, U19, U21, U35: 74HC04, Package_DIP:DIP-14_W7.62mm, symbol 74xx:74HC04
- removed U18: 74LS173, Package_DIP:DIP-16_W7.62mm, symbol 74xx:74LS173
- removed U20: 74LS244, symbol 74xx:74LS244
- removed U22: 74HCT244, symbol 74xx:74HCT244
- removed U9: M48T02-200PC1, Package_DIP:DIP-24_W15.24mm, symbol New_Library:M48T02-200PC1
- removed WD1: ~, symbol main-eagle-import:WD1770
- removed X1: ACO-10MHz, Oscillator:Oscillator_DIP-14, symbol Oscillator:ACO-xxxMHz
- removed X2: 8mhz_osc, Oscillator:Oscillator_DIP-14, symbol Oscillator:ACO-xxxMHz
- removed esp8266: ~, symbol Sol-1:esp8266
Connections:
- no-connect marks 162 -> 0
Other:
- sheet registers_paging renamed registers_paging_irq
- sheet registers_paging_irq: file registers_paging.kicad_sch -> registers_paging_irq.kicad_sch
- note removed: "0"
- note removed: "0 = kernel 1 = user"
- note removed: "000 = zf 001 = cf 010 = sf 011 = of 100 = s_l neg: s_ge 101 = s_le neg: s_g 001 = u_l neg: u_ge 110 = u_le neg: u_g"
- note removed: "1"
- note removed: "2"
- note removed: "244 microcode signals need inverter because they get reset to zero at beginning, and 244 are low active. this causes problems on reset."
- note removed: "3"
- note removed: "4"
- note removed: "5"
- note removed: "512kb ram modules. 8 modules giving a total of 4mb"
- note removed: "6"
- note removed: "7"
- note removed: "74HCT244 is used here because it recognizes TTL input levels. ttl levels are lower than CMOS, and the esp works at 3.3V. so when a high level is generated by the esp, it will go thru the HCT and it will trconize it as a high, whereas a niejjA"
- note removed: "74hc32 at ay20"
- note removed: "8253 TIMER"
- note removed: "HEAD LOAD (Option for double-sided version only) This signal line is used either HEAD LOAD or IN USE. When this signal is low, R/W head loads against the diskette. The set-up time of the solenoid is recuired before using this signal. This signal line responds to the input signal regardless of DRIVE SELECT line. IN USE (Option) When DRIVE SELECT signal is low, LOW level of this line will turn the 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"
- note removed: "IMPROVE THIS PART OF THE CIRCUIT"
- note removed: "M48T02 RTC"
- note removed: "NOT USED / NOT WIRED."
- note removed: "READY (Option) The LOW signal indicates that the diskette is rotating after properly inserted."
- note removed: "SIDE SELECT This signal defines which side of a two-sided diskette to be written on or read from. When this signal is LOW, side 1 head is selected, and when HIGH, side 0 head is selected. When switching from one side to the other, the waiting time is required before read/write operation starts."
- note removed: "These 3 signals are used in the memory decoder and hence show as dangling here."
- note removed: "a"
- note removed: "add mux here to create esc opcode"
- note removed: "adder"
- note removed: "alu"
- note removed: "alu output shifted by one"
- note removed: "alu_0 is what the carry flag becomes after a shift right alu_7 is what the cf becomes after a shift-left warning: this is not from the zbus~ this is before the alu's output is shifted~"
- note removed: "alu_0 is what the carry flag becomes after a shift right operation. warning: this is not from the zbus~ this is before the alu's output is shifted~"
- note removed: "alu_mode removed. of is undefined if alu in logic mode anyway."
- note removed: "alu_op == add"
- note removed: "alu_op == sub"
- note removed: "b"
- note removed: "bph"
- note removed: "bpl"
- note removed: "c"
- note removed: "carry in mux"
- note removed: "cf"
- note removed: "condition source programmer's flags or u_code flags"
- note removed: "d"
- note removed: "dih"
- note removed: "dil"
- note removed: "dma_ack is also used to tri-state the buses when in dma mode."
- note removed: "fdc input port"
- note removed: "fdc output port"
- note removed: "flags"
- note removed: "from wd1770"
- note removed: "front panel register display"
- note removed: "g_h"
- note removed: "g_l"
- note removed: "halt: use the halt flag to tri-state all buses. do microcode loop to test for interrupts or dma. if no interrupts or dma then just perform tight loop of zero offset. when int or dma appears, jump +1. next microinstr is pre-fetch type, so that int or dma can be executed. pc will be pointing to after halt. interrupts should always clear the halt flag, so that execution goes normally after the int f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"
- note removed: "high"
- note removed: "i need to add logic so that uart only activates if ad21 to ad16 are zero because that is the io area for when paging is on"
- note removed: "if fdc = 0, and a3 = 0, then we select this part of the fc bank, which is the part that contains the other config registers for the fdc."
- note removed: "if fdc is 0(enabled), and a3 is 1, we select the wd1770."
- note removed: "if type = branch, and condition = false, then next = +1"
- note removed: "int_pending input to conditional is to be used with halt instruction to check if ints are pending. it is also used with the cpu trace mode so that when coming out of the trace microcode loop, we can jump to the interrupts handler if interrupts are pending. without the int_pending conditional it is impossible to execute interrupts when executing in trace mode."
- note removed: "ir"
- note removed: "irq masks"
- note removed: "low"
- note removed: "lt lte ~lt = gte ~lte + gt"
- note removed: "marh"
- note removed: "marl"
- note removed: "mdr"
- note removed: "mdr mux"
- note removed: "microcode 0 to 63 is reserved for cpu startup. fetch at 0x10 trap at 0x20"
- note removed: "microcode sequencing"
- note removed: "might want to feed the external data bus directly into mar as well via a multiplexer. this is to speed-up ram operations"
- note removed: "of"
- note removed: "pch"
- note removed: "pcl"
- note removed: "ptb"
- note removed: "removed trace_mode flag from here. (no longer exists)"
- note removed: "rewiring the a1/a27 of the roms will be difficult and could damage the wiring and destroy the board."
- note removed: "select2 and select3 are permanently pulled HIGH. So drives 2 and 3 are not used."
- note removed: "sf"
- note removed: "shl: msb goes into cf. lsb replaced by 0 sla: same as shl rol: lsb becomes msb. rlc: msb goes into cf. lsb becomes cf shr: lsb goes into cf. msb replaced by 0 sra: lsb goes into cf. msb is whatever the previous one was ror: msb becomes lsb rrc: msb becomes cf. lsb goes into cf"
- note removed: "should add resistor here at clock select output because if clock floats, it could make stop_clock signal meta stable"
- note removed: "sih"
- note removed: "sil"
- note removed: "single step clock"
- note removed: "sph"
- note removed: "spl"
- note removed: "ssph"
- note removed: "sspl"
- note removed: "status"
- note removed: "tdr"
- note removed: "this 244 needs to be a flip flop instead, because the DRQ and READY lines are actually asynchronous."
- note removed: "this comes from the microcode board but is not a control bit. it is a combination of two bits."
- note removed: "this is the positive edge version of the master reset signal"
- note removed: "to calculate of when doing shifts we first save the sign of the original number, then when done shifting we save the value of the result. then we do a xor of both values, and the result is the of. the result of the xor is the msb of the result (zbus7). this is why wehave zbus7 as one of the inputs to of another possibility is to first save the sf into the u-flags register before doing the shifts,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"
- note removed: "typ1typ0 00 offset 01 branch 10 pre-fetch 11 post_fetch"
- note removed: "u-address"
- note removed: "u-address mux"
- note removed: "u_flags"
- note removed: "unused"
- note removed: "unused signals"
- note removed: "upper bits are a copy of u_offset6. this means this offset is a signed number from -64 to 63"
- note removed: "used for sign extension"
- note removed: "zf"
