File: hardware/schematics/kicad/memory_peripherals.kicad_sch (KiCad schematic)
At the start: 0 parts

Commit message: splitting schematic into blocks
Parts:
- added BIOS_ROM1: 27512, Package_DIP:DIP-28_W15.24mm, symbol main-eagle-import:27512
- added IC110, IC161, IC193, IC201: 74138N, Package_DIP:DIP-16_W7.62mm, symbol main-eagle-import:74138N
- added IC113, IC121, IC43: 7404N, Package_DIP:DIP-14_W7.62mm, symbol main-eagle-import:7404N
- added IC116: 74245N, Package_DIP:DIP-20_W7.62mm, symbol main-eagle-import:74245N
- added IC122: ~, main:DIL14, symbol main-eagle-import:7404N
- added IC162: 7420N, Package_DIP:DIP-14_W7.62mm, symbol main-eagle-import:7420N
- added IC165, IC35: 7408N, Package_DIP:DIP-14_W7.62mm, symbol main-eagle-import:7408N
- added IC171, IC188, IC192: 7432N, Package_DIP:DIP-14_W7.62mm, symbol main-eagle-import:7432N
- added IC172: 7430N, Package_DIP:DIP-14_W7.62mm, symbol main-eagle-import:7430N
- added IC173: 7427N, Package_DIP:DIP-14_W7.62mm, symbol main-eagle-import:7427N
- added IC174, IC176, IC195, IC199: 74244N, Package_DIP:DIP-20_W7.62mm, symbol main-eagle-import:74244N
- added IC189: ~, main:DIL14, symbol main-eagle-import:7432N
- added IC194: 74244N, Package_DIP:DIP-20_W7.62mm, symbol main-eagle-import:74xx-eu_74244N
- added IC86: ~, main:DIL14, symbol main-eagle-import:7408N
- added IC_10_1: 7410N, Package_DIP:DIP-14_W7.62mm, symbol main-eagle-import:7410N
- added J1: Conn_02x17_Odd_Even, symbol Connector_Generic:Conn_02x17_Odd_Even
- added PIO_1: 8255, Package_DIP:DIP-40_W15.24mm, symbol Interface:8255
- added RN9: R_Pack08, Package_DIP:DIP-16_W7.62mm, symbol Device:R_Pack08
- added U1, U2, U3, U4, U5, U6, U7, U8: as6c4008-55pcn, Package_DIP:DIP-32_W15.24mm, symbol main-eagle-import:AS6C4008-55PCN
- added U10, U9: 16550, Package_DIP:DIP-40_W15.24mm, symbol Interface_UART:16550
- added U11, U17: 74HC04, Package_DIP:DIP-14_W7.62mm, symbol 74xx:74HC04
- added U12: 74LS06, symbol 74xx:74LS06
- added U13: M48T02-200PC1, Package_DIP:DIP-24_W15.24mm, symbol New_Library:M48T02-200PC1
- added U14: 8253, Package_DIP:DIP-24_W15.24mm, symbol Timer:8253
- added U15: KM62256CLP, Package_DIP:DIP-28_W15.24mm, symbol Memory_RAM:KM62256CLP
- added U20: 74HCT244, symbol 74xx:74HCT244
- added U21: 74LS377, symbol 74xx:74LS377
- added U22: 74LS244, symbol 74xx:74LS244
- added WD1: ~, symbol main-eagle-import:WD1770
- added X2: 8mhz_osc, Oscillator:Oscillator_DIP-14, symbol Oscillator:ACO-xxxMHz
- added esp1: ~, symbol Sol-1:esp8266
Connections:
- new net: BIOS_ROM1.27 (A14), IC172.1 (I0), IC176.5 (Y3), U15.1 (A14)
- new net: BIOS_ROM1.25 (A8), IC172.11 (I6), IC176.18 (Y1), U15.25 (A8)
- new net: BIOS_ROM1.3 (A7), IC172.12 (I7), IC174.3 (Y4), U15.3 (A7)
- new net: BIOS_ROM1.26 (A13), IC172.2 (I1), IC176.7 (Y2), U15.26 (A13)
- new net: BIOS_ROM1.2 (A12), IC172.3 (I2), IC176.9 (Y1), U15.2 (A12)
- new net: BIOS_ROM1.23 (A11), IC172.4 (I3), IC176.12 (Y4), U15.23 (A11)
- new net: BIOS_ROM1.21 (A10), IC172.5 (I4), IC176.14 (Y3), U15.21 (A10)
- new net: BIOS_ROM1.24 (A9), IC172.6 (I5), IC176.16 (Y2), U15.24 (A9)
- new net: IC121.4 (O), IC35.5 (I1)
- new net: IC188.6 (O), IC43.3 (I)
- new net: U20.2 (1A0), esp1.1 (tx)
- new net: BIOS_ROM1.10 (A0), IC174.18 (Y1), U15.10 (A0)
- new net: BIOS_ROM1.11 (O0), IC116.18 (B1), U15.11 (Q0)
- new net: BIOS_ROM1.12 (O1), IC116.17 (B2), U15.12 (Q1)
- new net: BIOS_ROM1.13 (O2), IC116.16 (B3), U15.13 (Q2)
- new net: BIOS_ROM1.15 (O3), IC116.15 (B4), U15.15 (Q3)
- new net: BIOS_ROM1.16 (O4), IC116.14 (B5), U15.16 (Q4)
- new net: BIOS_ROM1.17 (O5), IC116.13 (B6), U15.17 (Q5)
- new net: BIOS_ROM1.18 (O6), IC116.12 (B7), U15.18 (Q6)
- new net: BIOS_ROM1.19 (O7), IC116.11 (B8), U15.19 (Q7)
- new net: BIOS_ROM1.20 (~{CE}), IC_10_1.8 (O)
- new net: BIOS_ROM1.4 (A6), IC161.3 (C), IC174.5 (Y3), U15.4 (A6)
- new net: BIOS_ROM1.5 (A5), IC161.2 (B), IC174.7 (Y2), U15.5 (A5)
- new net: BIOS_ROM1.6 (A4), IC161.1 (A), IC174.9 (Y1), U15.6 (A4)
- new net: BIOS_ROM1.7 (A3), IC110.1 (A), IC174.12 (Y4), U15.7 (A3)
- new net: BIOS_ROM1.8 (A2), IC174.14 (Y3), U15.8 (A2)
- new net: BIOS_ROM1.9 (A1), IC174.16 (Y2), U15.9 (A1)
- new net: IC173.5 (I2), IC199.12 (Y4), IC201.1 (A)
- new net: IC173.4 (I1), IC199.9 (Y1), IC201.2 (B)
- new net: IC173.3 (I0), IC199.7 (Y2), IC201.3 (C)
- new net: IC165.1 (I0), IC173.6 (O)
- new net: IC165.2 (I1), IC173.12 (O)
- new net: IC162.2 (I1), IC165.3 (O), IC_10_1.10 (I1)
- new net: IC113.1 (I), IC162.5 (I3), IC176.3 (Y4), IC35.4 (I0)
- new net: IC162.6 (O), U15.20 (~{CS})
- new net: IC171.3 (O), IC189.1 (I0)
- new net: IC189.2 (I1), IC86.3 (O)
- new net: IC189.3 (O), WD1.1 (~{CS})
- new net: U12.11, WD1.16 (STEP)
- new net: IC194.4 (A2), U17.2
- new net: IC173.1 (I0), IC199.14 (Y3)
- new net: IC173.2 (I1), IC199.16 (Y2)
- new net: IC173.13 (I2), IC199.18 (Y1)
- new net: IC194.2 (A1), U17.4
- new net: IC171.8 (O), U22.1 (OEa), U22.19 (OEb)
- new net: U12.3, WD1.21 (WG)
- new net: U12.9, WD1.17 (DIRC)
- new net: IC161.6 (G1), IC35.6 (O)
- new net: IC113.2 (O), IC_10_1.9 (I0)
- new net: U12.5, WD1.20 (MO)
- new net: IC110.6 (G1), IC122.2 (O)
- new net: IC122.1 (I), IC161.15 (Y0)
- new net: IC113.6 (O), IC161.4 (G2A), IC161.5 (G2B)
- new net: IC43.4 (O), WD1.13 (~{MR})
- new net: U12.1, WD1.22 (WD)
- new net: IC171.6 (O), U21.1 (~{E})
- new net: IC171.1 (I0), U11.2
- new net GND: BIOS_ROM1.1 (A15), IC110.2 (B), IC110.3 (C), IC110.4 (G2A), IC110.5 (G2B), IC116.19 (G), IC174.1 (G), IC174.19 (G), IC176.1 (G), IC176.19 (G), IC194.6 (A3), IC194.8 (A4), IC195.1 (G), IC195.13 (A2), IC195.15 (A3), IC195.17 (A4), IC195.19 (G), IC199.1 (G), IC199.15 (A3), IC199.17 (A4), IC199.19 (G), J1.1 (Pin_1), J1.11 (Pin_11), J1.13 (Pin_13), J1.15 (Pin_15), J1.17 (Pin_17), J1.19 (Pin_19), J1.21 (Pin_21), J1.23 (Pin_23), J1.25 (Pin_25), J1.27 (Pin_27), J1.29 (Pin_29), J1.3 (Pin_3), J1.31 (Pin_31), J1.33 (Pin_33), J1.5 (Pin_5), J1.7 (Pin_7), J1.9 (Pin_9), PIO_1.7 (GND), U1.16 (VSS), U10.12 (CS0), U10.13 (CS1), U10.19 (WR), U10.20 (GND), U10.22 (RD), U13.12 (GND), U14.12 (GND), U15.14 (GND), U2.16 (VSS), U3.16 (VSS), U4.16 (VSS), U5.16 (VSS), U6.16 (VSS), U7.16 (VSS), U8.16 (VSS), U9.12 (CS0), U9.13 (CS1), U9.19 (WR), U9.20 (GND), U9.22 (RD), WD1.14 (GND), X2.7 (GND)
- new net VCC: IC193.6 (G1), J1.14 (Pin_14), J1.6 (Pin_6), PIO_1.26 (VCC), RN9.1 (R1.1), RN9.2 (R2.1), RN9.3 (R3.1), RN9.4 (R4.1), RN9.5 (R5.1), RN9.6 (R6.1), RN9.7 (R7.1), RN9.8 (R8.1), U1.32 (VCC), U10.40 (VCC), U13.24 (VCC), U14.24 (VCC), U15.28 (VCC), U2.32 (VCC), U3.32 (VCC), U4.32 (VCC), U5.32 (VCC), U6.32 (VCC), U7.32 (VCC), U8.32 (VCC), U9.40 (VCC), WD1.15 (VCC)
- new net a0: IC193.1 (A)
- new net a1: IC193.2 (B)
- new net a2: IC193.3 (C)
- new net a3: IC193.4 (G2A), U11.1
- new net address_bus0: IC174.2 (A1), PIO_1.9 (A0), U1.12 (A0), U10.28 (A0), U13.1 (A7), U14.19 (A0), U2.12 (A0), U3.12 (A0), U4.12 (A0), U5.12 (A0), U6.12 (A0), U7.12 (A0), U8.12 (A0), U9.28 (A0), WD1.3 (A0)
- new net address_bus1: IC174.4 (A2), PIO_1.8 (A1), U1.11 (A1), U10.27 (A1), U13.2 (A6), U14.20 (A1), U2.11 (A1), U3.11 (A1), U4.11 (A1), U5.11 (A1), U6.11 (A1), U7.11 (A1), U8.11 (A1), U9.27 (A1), WD1.4 (A1)
- new net address_bus10: IC176.6 (A3), U1.23 (A10), U13.19 (A10), U2.23 (A10), U3.23 (A10), U4.23 (A10), U5.23 (A10), U6.23 (A10), U7.23 (A10), U8.23 (A10)
- new net address_bus11: IC176.8 (A4), U1.25 (A11), U2.25 (A11), U3.25 (A11), U4.25 (A11), U5.25 (A11), U6.25 (A11), U7.25 (A11), U8.25 (A11)
- new net address_bus12: IC176.11 (A1), U1.4 (A12), U2.4 (A12), U3.4 (A12), U4.4 (A12), U5.4 (A12), U6.4 (A12), U7.4 (A12), U8.4 (A12)
- new net address_bus13: IC176.13 (A2), U1.28 (A13), U2.28 (A13), U3.28 (A13), U4.28 (A13), U5.28 (A13), U6.28 (A13), U7.28 (A13), U8.28 (A13)
- new net address_bus14: IC176.15 (A3), U1.3 (A14), U2.3 (A14), U3.3 (A14), U4.3 (A14), U5.3 (A14), U6.3 (A14), U7.3 (A14), U8.3 (A14)
- new net address_bus15: IC176.17 (A4), U1.31 (A15), U2.31 (A15), U3.31 (A15), U4.31 (A15), U5.31 (A15), U6.31 (A15), U7.31 (A15), U8.31 (A15)
- new net address_bus16: IC199.2 (A1), U1.2 (A16), U2.2 (A16), U3.2 (A16), U4.2 (A16), U5.2 (A16), U6.2 (A16), U7.2 (A16), U8.2 (A16)
- new net address_bus17: IC199.4 (A2), U1.30 (A17), U2.30 (A17), U3.30 (A17), U4.30 (A17), U5.30 (A17), U6.30 (A17), U7.30 (A17), U8.30 (A17)
- new net address_bus18: IC199.6 (A3), U1.1 (A18), U2.1 (A18), U3.1 (A18), U4.1 (A18), U5.1 (A18), U6.1 (A18), U7.1 (A18), U8.1 (A18)
- new net address_bus19: IC199.8 (A4)
- new net address_bus2: IC174.6 (A3), U1.10 (A2), U10.26 (A2), U13.3 (A5), U2.10 (A2), U3.10 (A2), U4.10 (A2), U5.10 (A2), U6.10 (A2), U7.10 (A2), U8.10 (A2), U9.26 (A2)
- new net address_bus20: IC199.11 (A1)
- new net address_bus21: IC199.13 (A2)
- new net address_bus3: IC174.8 (A4), U1.9 (A3), U13.4 (A4), U2.9 (A3), U3.9 (A3), U4.9 (A3), U5.9 (A3), U6.9 (A3), U7.9 (A3), U8.9 (A3)
- new net address_bus4: IC174.11 (A1), U1.8 (A4), U13.5 (A3), U2.8 (A4), U3.8 (A4), U4.8 (A4), U5.8 (A4), U6.8 (A4), U7.8 (A4), U8.8 (A4)
- new net address_bus5: IC174.13 (A2), U1.7 (A5), U13.6 (A2), U2.7 (A5), U3.7 (A5), U4.7 (A5), U5.7 (A5), U6.7 (A5), U7.7 (A5), U8.7 (A5)
- new net address_bus6: IC174.15 (A3), U1.6 (A6), U13.7 (A1), U2.6 (A6), U3.6 (A6), U4.6 (A6), U5.6 (A6), U6.6 (A6), U7.6 (A6), U8.6 (A6)
- new net address_bus7: IC174.17 (A4), U1.5 (A7), U13.8 (A0), U2.5 (A7), U3.5 (A7), U4.5 (A7), U5.5 (A7), U6.5 (A7), U7.5 (A7), U8.5 (A7)
- new net address_bus8: IC176.2 (A1), U1.27 (A8), U13.23 (A8), U2.27 (A8), U3.27 (A8), U4.27 (A8), U5.27 (A8), U6.27 (A8), U7.27 (A8), U8.27 (A8)
- new net address_bus9: IC176.4 (A2), U1.26 (A9), U13.22 (A9), U2.26 (A9), U3.26 (A9), U4.26 (A9), U5.26 (A9), U6.26 (A9), U7.26 (A9), U8.26 (A9)
- new net bios_config: IC161.7 (Y7)
- new net buffered_mem_io: IC113.5 (I), IC162.1 (I0), IC195.14 (Y3), IC201.4 (G2A), IC201.5 (G2B), IC_10_1.11 (I2)
- new net buffered_rd: BIOS_ROM1.22 (~{OE}), IC116.1 (DIR), IC171.10 (I1), IC195.18 (Y1), IC86.1 (I0), PIO_1.5 (~{RD}), U10.21 (~{RD}), U13.20 (*OE), U14.22 (~{RD}), U15.22 (~{OE}), U9.21 (~{RD})
- new net buffered_rd_memory: IC195.12 (Y4), U1.24 (OE), U2.24 (OE), U3.24 (OE), U4.24 (OE), U5.24 (OE), U6.24 (OE), U7.24 (OE), U8.24 (OE)
- new net buffered_wr: IC171.5 (I1), IC195.16 (Y2), IC86.2 (I1), PIO_1.36 (~{WR}), U10.18 (~{WR}), U13.21 (*WE), U14.23 (~{WR}), U15.27 (~{WE}), U9.18 (~{WR}), WD1.2 (R/~{W})
- new net buffered_wr_memory: IC195.9 (Y1), U1.29 (WE), U2.29 (WE), U3.29 (WE), U4.29 (WE), U5.29 (WE), U6.29 (WE), U7.29 (WE), U8.29 (WE)
- new net bus_mem_io: IC195.6 (A3)
- new net bus_rd: IC194.18 (Y1), IC195.2 (A1), IC195.8 (A4)
- new net bus_tristate: IC121.9 (I), IC192.6 (O), IC194.1 (G)
- new net bus_wr: IC194.16 (Y2), IC195.11 (A1), IC195.4 (A2)
- new net clk: U21.11 (CP)
- new net clk_8mhz: WD1.18 (CLK), X2.8 (OUT)
- new net data_bus0: IC116.2 (A1), PIO_1.34 (D0), U1.13 (DQ0), U10.1 (D0), U13.9 (DQ0), U14.8 (D0), U2.13 (DQ0), U21.3 (D0), U22.18 (O0a), U3.13 (DQ0), U4.13 (DQ0), U5.13 (DQ0), U6.13 (DQ0), U7.13 (DQ0), U8.13 (DQ0), U9.1 (D0), WD1.5 (DAL0)
- new net data_bus1: IC116.3 (A2), PIO_1.33 (D1), U1.14 (DQ1), U10.2 (D1), U13.10 (DQ1), U14.7 (D1), U2.14 (DQ1), U21.4 (D1), U22.16 (O1a), U3.14 (DQ1), U4.14 (DQ1), U5.14 (DQ1), U6.14 (DQ1), U7.14 (DQ1), U8.14 (DQ1), U9.2 (D1), WD1.6 (DAL1)
- new net data_bus2: IC116.4 (A3), PIO_1.32 (D2), U1.15 (DQ2), U10.3 (D2), U13.11 (DQ2), U14.6 (D2), U2.15 (DQ2), U21.7 (D2), U22.14 (O2a), U3.15 (DQ2), U4.15 (DQ2), U5.15 (DQ2), U6.15 (DQ2), U7.15 (DQ2), U8.15 (DQ2), U9.3 (D2), WD1.7 (DAL2)
- new net data_bus3: IC116.5 (A4), PIO_1.31 (D3), U1.17 (DQ3), U10.4 (D3), U13.13 (DQ3), U14.5 (D3), U2.17 (DQ3), U21.8 (D3), U22.12 (O3a), U3.17 (DQ3), U4.17 (DQ3), U5.17 (DQ3), U6.17 (DQ3), U7.17 (DQ3), U8.17 (DQ3), U9.4 (D3), WD1.8 (DAL3)
- new net data_bus4: IC116.6 (A5), PIO_1.30 (D4), U1.18 (DQ4), U10.5 (D4), U13.14 (DQ4), U14.4 (D4), U2.18 (DQ4), U21.13 (D4), U22.9 (O0b), U3.18 (DQ4), U4.18 (DQ4), U5.18 (DQ4), U6.18 (DQ4), U7.18 (DQ4), U8.18 (DQ4), U9.5 (D4), WD1.9 (DAL4)
- new net data_bus5: IC116.7 (A6), PIO_1.29 (D5), U1.19 (DQ5), U10.6 (D5), U13.15 (DQ5), U14.3 (D5), U2.19 (DQ5), U21.14 (D5), U22.7 (O1b), U3.19 (DQ5), U4.19 (DQ5), U5.19 (DQ5), U6.19 (DQ5), U7.19 (DQ5), U8.19 (DQ5), U9.6 (D5), WD1.10 (DAL5)
- new net data_bus6: IC116.8 (A7), PIO_1.28 (D6), U1.20 (DQ6), U10.7 (D6), U13.16 (DQ6), U14.2 (D6), U2.20 (DQ6), U21.17 (D6), U22.5 (O2b), U3.20 (DQ6), U4.20 (DQ6), U5.20 (DQ6), U6.20 (DQ6), U7.20 (DQ6), U8.20 (DQ6), U9.7 (D6), WD1.11 (DAL6)
- new net data_bus7: IC116.9 (A8), PIO_1.27 (D7), U1.21 (DQ7), U10.8 (D7), U13.17 (DQ7), U14.1 (D7), U2.21 (DQ7), U21.18 (D7), U22.3 (O3b), U3.21 (DQ7), U4.21 (DQ7), U5.21 (DQ7), U6.21 (DQ7), U7.21 (DQ7), U8.21 (DQ7), U9.8 (D7), WD1.12 (DAL7)
- new net dir: J1.18 (Pin_18), U12.8
- new net double_density_en: PIO_1.21 (PB3), U21.9 (Q3), WD1.26 (~{DDEN})
- new net fdc: IC161.11 (Y4), IC171.2 (I1), IC193.5 (G2B)
- new net fdc_drq: PIO_1.4 (PA0), U22.2 (I0a), WD1.27 (DRQ)
- new net fdc_input_port_re: IC171.9 (I0), IC193.14 (Y1)
- new net fdc_irq: WD1.28 (INTRQ)
- new net fdc_output_port_we: IC171.4 (I0), IC193.15 (Y0)
- new net ide_en: IC161.10 (Y5)
- new net in_use_or_head_load: J1.4 (Pin_4), PIO_1.22 (PB4), U21.12 (Q4)
- new net index: J1.8 (Pin_8), RN9.15 (R2.2), WD1.24 (~{IP})
- new net irq0: U10.30 (INTR)
- new net irq1: U9.30 (INTR)
- new net mem_select_0: IC201.15 (Y0), U7.22 (CE)
- new net mem_select_1: IC201.14 (Y1), U6.22 (CE)
- new net mem_select_2: IC201.13 (Y2), U5.22 (CE)
- new net mem_select_3: IC201.12 (Y3), U4.22 (CE)
- new net mem_select_4: IC201.11 (Y4), U8.22 (CE)
- new net mem_select_5: IC201.10 (Y5), U3.22 (CE)
- new net mem_select_6: IC201.9 (Y6), U2.22 (CE)
- new net mem_select_7: IC201.7 (Y7), U1.22 (CE)
- new net motor_en: J1.16 (Pin_16), U12.6
- new net pio_0_en: IC161.12 (Y3), PIO_1.6 (~{CS})
- new net rd: U17.3
- new net read_data: J1.30 (Pin_30), RN9.13 (R4.2), WD1.19 (~{RD})
- new net ready: J1.34 (Pin_34), RN9.12 (R5.2), U22.4 (I1a)
- new net rst: IC188.4 (I0)
- new net rtc_en: IC161.13 (Y2), U13.18 (*CE)
- new net select_0: J1.10 (Pin_10), PIO_1.18 (PB0), U21.2 (Q0)
- new net select_1: J1.12 (Pin_12), PIO_1.19 (PB1), U21.5 (Q1)
- new net side_select: J1.32 (Pin_32), PIO_1.20 (PB2), U21.6 (Q2)
- new net status_dma_ack: IC192.4 (I0)
- new net status_halt: IC192.5 (I1)
- new net step: J1.20 (Pin_20), U12.10
- new net timer_en: IC161.9 (Y6), U14.21 (~{CS})
- new net track_0: J1.26 (Pin_26), RN9.14 (R3.2), WD1.23 (~{TR00})
- new net uart_0_en: IC110.15 (Y0), U10.14 (~{CS2})
- new net uart_0_rx_pin: U10.10 (SIN), U20.18 (1Y0)
- new net uart_1_en: IC110.14 (Y1), U9.14 (~{CS2})
- new net vcc: IC201.6 (G1), X2.14 (Vcc)
- new net wd1770_rst: IC188.5 (I1), U21.15 (Q5)
- new net wr: U17.1
- new net write_data: J1.22 (Pin_22), U12.2
- new net write_gate: J1.24 (Pin_24), U12.4
- new net write_protect: J1.28 (Pin_28), RN9.16 (R1.2), WD1.25 (~{WPRT})
- new net ~{addr_bus_7_to_14_alltrue}: IC121.3 (I), IC162.4 (I2), IC172.8 (O)
- new net ~{bus_tristate}: IC121.8 (O)
- new net ~{ready}: PIO_1.3 (PA1)
- no-connect marks 0 -> 28
Other:
- note added: "512kb ram modules. 8 modules giving a total of 4mb"
- note added: "74HCT244 is used here because it recognizes TTL input levels. ttl levels are lower than CMOS, and the esp works at 3.3V. so when a high level is generated by the esp, it will go thru the HCT and it will trconize it as a high, whereas a niejjA"
- note added: "8253 TIMER"
- note added: "HEAD LOAD (Option for double-sided version only) This signal line is used either HEAD LOAD or IN USE. When this signal is low, R/W head loads against the diskette. The set-up time of the solenoid is recuired before using this signal. This signal line responds to the input signal regardless of DRIVE SELECT line. IN USE (Option) When DRIVE SELECT signal is low, LOW level of this line will turn the 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"
- note added: "M48T02 RTC"
- note added: "NOT USED / NOT WIRED."
- note added: "READY (Option) The LOW signal indicates that the diskette is rotating after properly inserted."
- note added: "SIDE SELECT This signal defines which side of a two-sided diskette to be written on or read from. When this signal is LOW, side 1 head is selected, and when HIGH, side 0 head is selected. When switching from one side to the other, the waiting time is required before read/write operation starts."
- note added: "These 3 signals are used in the memory decoder and hence show as dangling here."
- note added: "fdc input port"
- note added: "fdc output port"
- note added: "from wd1770"
- note added: "i need to add logic so that uart only activates if ad21 to ad16 are zero because that is the io area for when paging is on"
- note added: "if fdc = 0, and a3 = 0, then we select this part of the fc bank, which is the part that contains the other config registers for the fdc."
- note added: "if fdc is 0(enabled), and a3 is 1, we select the wd1770."
- note added: "select2 and select3 are permanently pulled HIGH. So drives 2 and 3 are not used."
- note added: "this 244 needs to be a flip flop instead, because the DRQ and READY lines are actually asynchronous."
- note added: "this is the positive edge version of the master reset signal"
