File: hardware/schematics/kicad/microcode_alu.kicad_sch (KiCad schematic)
At the start: 0 parts

Commit message: splitting schematic into blocks
Parts:
- added ALU_HIGH1, ALU_LOW1: 74181N, Package_DIP:DIP-24_W7.62mm, symbol main-eagle-import:74181N
- added C1: C, Capacitor_THT:C_Disc_D7.5mm_W4.4mm_P5.00mm, symbol Device:C
- added FLAGS1, IC100, IC101, IC102, IC103, IC104, IC105, IC106, IC107, IC108, IC22, IC91, IC92, IC94, IC95, IC96, IC97, IC98, IC99: 74273N, Package_DIP:DIP-20_W7.62mm, symbol main-eagle-import:74273N
- added IC1, IC2, IC36, IC42: 74377N, Package_DIP:DIP-20_W7.62mm, symbol main-eagle-import:74377N
- added IC10, IC14, IC17, IC18, IC66, IC68, IC7, IC77, IC78, IC79, IC8, IC80, IC81, IC82, IC83, IC9: 74153N, Package_DIP:DIP-16_W7.62mm, symbol main-eagle-import:74153N
- added IC11, IC12, IC15, IC16, IC19, IC20, IC24, IC25, IC26, IC27, IC30, IC76, IC89: 74257N, Package_DIP:DIP-16_W7.62mm, symbol main-eagle-import:74257N
- added IC13, IC35: 7408N, Package_DIP:DIP-14_W7.62mm, symbol main-eagle-import:7408N
- added IC21: 7404N, Package_DIP:DIP-14_W7.62mm, symbol main-eagle-import:7404N
- added IC23, IC_10_1: 7410N, Package_DIP:DIP-14_W7.62mm, symbol main-eagle-import:7410N
- added IC28, IC49, IC50, IC67, IC69: 74151N, Package_DIP:DIP-16_W7.62mm, symbol main-eagle-import:74151N
- added IC29, IC44, IC45, IC48: 7432N, Package_DIP:DIP-14_W7.62mm, symbol main-eagle-import:7432N
- added IC3, IC31, IC32, IC33, IC34, IC4, IC5, IC6: 74253N, Package_DIP:DIP-16_W7.62mm, symbol main-eagle-import:74253N
- added IC37, IC_86_1, IC_86_2: 7486N, Package_DIP:DIP-14_W7.62mm, symbol main-eagle-import:7486N
- added IC38, IC39, IC40, IC41: 74283N, Package_DIP:DIP-16_W7.62mm, symbol main-eagle-import:74283N
- added IC47: 74244N, Package_DIP:DIP-20_W7.62mm, symbol main-eagle-import:74xx-eu_74244N
- added IC51: 7427N, Package_DIP:DIP-14_W7.62mm, symbol main-eagle-import:7427N
- added IC65: 7411N, Package_DIP:DIP-14_W7.62mm, symbol main-eagle-import:7411N
- added IC_02_1: 7402N, Package_DIP:DIP-14_W7.62mm, symbol main-eagle-import:7402N
- added IC_04_1: 7404N, Package_DIP:DIP-14_W7.62mm, symbol main-eagle-import:74xx-eu_7404N
- added U_ROM1, U_ROM10, U_ROM11, U_ROM12, U_ROM13, U_ROM14, U_ROM15, U_ROM2, U_ROM3, U_ROM4, U_ROM5, U_ROM6, U_ROM7, U_ROM8, U_ROM9: 27512, Package_DIP:DIP-28_W15.24mm, symbol main-eagle-import:27512
Connections:
- new net: IC25.12 (4Y), IC39.11 (B4)
- new net: IC25.9 (3Y), IC39.15 (B3)
- new net: IC25.7 (2Y), IC39.2 (B2)
- new net: IC25.4 (1Y), IC39.6 (B1)
- new net: IC38.9 (C4), IC39.7 (C0)
- new net: IC39.9 (C4), IC40.7 (C0)
- new net: IC98.3 (D1), U_ROM5.11 (O0)
- new net: IC98.4 (D2), U_ROM5.12 (O1)
- new net: IC98.7 (D3), U_ROM5.13 (O2)
- new net: IC98.8 (D4), U_ROM5.15 (O3)
- new net: IC98.13 (D5), U_ROM5.16 (O4)
- new net: IC98.14 (D6), U_ROM5.17 (O5)
- new net: IC98.17 (D7), U_ROM5.18 (O6)
- new net: IC98.18 (D8), U_ROM5.19 (O7)
- new net: IC105.3 (D1), U_ROM12.11 (O0)
- new net: IC105.4 (D2), U_ROM12.12 (O1)
- new net: IC105.7 (D3), U_ROM12.13 (O2)
- new net: IC105.8 (D4), U_ROM12.15 (O3)
- new net: IC105.13 (D5), U_ROM12.16 (O4)
- new net: IC105.14 (D6), U_ROM12.17 (O5)
- new net: IC105.17 (D7), U_ROM12.18 (O6)
- new net: IC105.18 (D8), U_ROM12.19 (O7)
- new net: IC106.3 (D1), U_ROM13.11 (O0)
- new net: IC106.4 (D2), U_ROM13.12 (O1)
- new net: IC106.7 (D3), U_ROM13.13 (O2)
- new net: IC106.8 (D4), U_ROM13.15 (O3)
- new net: IC106.13 (D5), U_ROM13.16 (O4)
- new net: IC106.14 (D6), U_ROM13.17 (O5)
- new net: IC106.17 (D7), U_ROM13.18 (O6)
- new net: IC106.18 (D8), U_ROM13.19 (O7)
- new net: IC17.7 (1Y), IC22.3 (D1)
- new net: IC18.7 (1Y), IC22.4 (D2)
- new net: IC19.4 (1Y), IC22.7 (D3)
- new net: IC20.4 (1Y), IC22.8 (D4)
- new net: IC49.5 (Y), IC76.2 (1A)
- new net: IC50.5 (Y), IC76.3 (1B)
- new net: IC77.7 (1Y), IC91.3 (D1)
- new net: IC77.9 (2Y), IC91.4 (D2)
- new net: IC99.3 (D1), U_ROM6.11 (O0)
- new net: IC99.4 (D2), U_ROM6.12 (O1)
- new net: IC99.7 (D3), U_ROM6.13 (O2)
- new net: IC99.8 (D4), U_ROM6.15 (O3)
- new net: IC99.13 (D5), U_ROM6.16 (O4)
- new net: IC99.14 (D6), U_ROM6.17 (O5)
- new net: IC99.17 (D7), U_ROM6.18 (O6)
- new net: IC99.18 (D8), U_ROM6.19 (O7)
- new net: IC51.8 (O), IC65.13 (I2)
- new net: IC78.7 (1Y), IC91.7 (D3)
- new net: IC78.9 (2Y), IC91.8 (D4)
- new net: IC108.3 (D1), U_ROM15.11 (O0)
- new net: IC108.4 (D2), U_ROM15.12 (O1)
- new net: IC108.7 (D3), U_ROM15.13 (O2)
- new net: IC108.8 (D4), U_ROM15.15 (O3)
- new net: IC108.13 (D5), U_ROM15.16 (O4)
- new net: IC108.14 (D6), U_ROM15.17 (O5)
- new net: IC108.17 (D7), U_ROM15.18 (O6)
- new net: IC108.18 (D8), U_ROM15.19 (O7)
- new net: IC103.3 (D1), U_ROM10.11 (O0)
- new net: IC103.4 (D2), U_ROM10.12 (O1)
- new net: IC103.7 (D3), U_ROM10.13 (O2)
- new net: IC103.8 (D4), U_ROM10.15 (O3)
- new net: IC103.13 (D5), U_ROM10.16 (O4)
- new net: IC103.14 (D6), U_ROM10.17 (O5)
- new net: IC103.17 (D7), U_ROM10.18 (O6)
- new net: IC103.18 (D8), U_ROM10.19 (O7)
- new net: IC96.3 (D1), U_ROM3.11 (O0)
- new net: IC96.4 (D2), U_ROM3.12 (O1)
- new net: IC96.7 (D3), U_ROM3.13 (O2)
- new net: IC96.8 (D4), U_ROM3.15 (O3)
- new net: IC96.13 (D5), U_ROM3.16 (O4)
- new net: IC96.14 (D6), U_ROM3.17 (O5)
- new net: IC96.17 (D7), U_ROM3.18 (O6)
- new net: IC96.18 (D8), U_ROM3.19 (O7)
- new net: IC1.19 (8Q), IC6.12 (2C2)
- new net: IC2.19 (8Q), IC6.13 (2C3)
- new net: IC2.16 (7Q), IC6.3 (1C3)
- new net: IC1.16 (7Q), IC6.4 (1C2)
- new net: IC12.10 (3B), IC6.7 (1Y)
- new net: IC12.13 (4B), IC6.9 (2Y)
- new net: IC30.12 (4Y), IC37.5 (I1), IC49.1 (D3)
- new net: IC30.4 (1Y), IC44.5 (I1), IC45.5 (I1), IC49.4 (D0)
- new net: IC30.7 (2Y), IC45.4 (I0), IC49.3 (D1)
- new net: IC30.9 (3Y), IC37.4 (I0), IC49.2 (D2)
- new net: IC51.6 (O), IC65.2 (I1)
- new net: IC101.3 (D1), U_ROM8.11 (O0)
- new net: IC101.4 (D2), U_ROM8.12 (O1)
- new net: IC101.7 (D3), U_ROM8.13 (O2)
- new net: IC101.8 (D4), U_ROM8.15 (O3)
- new net: IC101.13 (D5), U_ROM8.16 (O4)
- new net: IC101.14 (D6), U_ROM8.17 (O5)
- new net: IC101.17 (D7), U_ROM8.18 (O6)
- new net: IC101.18 (D8), U_ROM8.19 (O7)
- new net: IC11.10 (3B), IC4.7 (1Y)
- new net: IC11.13 (4B), IC4.9 (2Y)
- new net: IC11.3 (1B), IC3.7 (1Y)
- new net: IC11.6 (2B), IC3.9 (2Y)
- new net: IC_10_1.3 (I0), IC_86_2.3 (O)
- new net: IC95.3 (D1), U_ROM2.11 (O0)
- new net: IC95.4 (D2), U_ROM2.12 (O1)
- new net: IC95.7 (D3), U_ROM2.13 (O2)
- new net: IC95.8 (D4), U_ROM2.15 (O3)
- new net: IC95.13 (D5), U_ROM2.16 (O4)
- new net: IC95.14 (D6), U_ROM2.17 (O5)
- new net: IC95.17 (D7), U_ROM2.18 (O6)
- new net: IC95.18 (D8), U_ROM2.19 (O7)
- new net: IC83.7 (1Y), IC92.13 (D5)
- new net: IC83.9 (2Y), IC92.14 (D6)
- new net: IC81.7 (1Y), IC92.3 (D1)
- new net: IC81.9 (2Y), IC92.4 (D2)
- new net: IC82.7 (1Y), IC92.7 (D3)
- new net: IC82.9 (2Y), IC92.8 (D4)
- new net: FLAGS1.7 (D3), IC68.7 (1Y)
- new net: IC37.6 (O), IC44.4 (I0), IC49.15 (D4)
- new net: IC79.7 (1Y), IC91.13 (D5)
- new net: IC79.9 (2Y), IC91.14 (D6)
- new net: IC_86_2.10 (I1), IC_86_2.6 (O)
- new net: IC_04_1.1 (I), IC_86_2.8 (O)
- new net: IC_10_1.12 (O), IC_86_2.9 (I0)
- new net: IC_02_1.1 (O), IC_10_1.13 (I2)
- new net: IC_04_1.2 (O), IC_10_1.5 (I2)
- new net: IC_04_1.3 (I), IC_10_1.6 (O)
- new net: IC65.6 (O), IC66.4 (1C2)
- new net: FLAGS1.18 (D8), IC89.12 (4Y)
- new net: FLAGS1.13 (D5), IC89.4 (1Y)
- new net: FLAGS1.14 (D6), IC89.7 (2Y)
- new net: FLAGS1.17 (D7), IC89.9 (3Y)
- new net: IC100.13 (D5), U_ROM7.16 (O4)
- new net: IC100.14 (D6), U_ROM7.17 (O5)
- new net: IC100.17 (D7), U_ROM7.18 (O6)
- new net: IC100.18 (D8), U_ROM7.19 (O7)
- new net: IC100.3 (D1), U_ROM7.11 (O0)
- new net: IC100.4 (D2), U_ROM7.12 (O1)
- new net: IC100.7 (D3), U_ROM7.13 (O2)
- new net: IC100.8 (D4), U_ROM7.15 (O3)
- new net: IC21.2 (O), IC23.2 (I1)
- new net: IC31.7 (1Y), IC47.2 (A1)
- new net: IC31.9 (2Y), IC47.4 (A2)
- new net: IC32.7 (1Y), IC47.6 (A3)
- new net: IC32.9 (2Y), IC47.8 (A4)
- new net: IC13.5 (I1), IC13.9 (I0), IC21.8 (O)
- new net: IC69.15 (D4), IC_86_1.8 (O)
- new net: FLAGS1.3 (D1), IC66.7 (1Y)
- new net: FLAGS1.4 (D2), IC67.5 (Y)
- new net: FLAGS1.8 (D4), IC69.5 (Y)
- new net: IC1.15 (6Q), IC5.12 (2C2)
- new net: IC2.15 (6Q), IC5.13 (2C3)
- new net: IC2.12 (5Q), IC5.3 (1C3)
- new net: IC1.12 (5Q), IC5.4 (1C2)
- new net: IC12.3 (1B), IC5.7 (1Y)
- new net: IC12.6 (2B), IC5.9 (2Y)
- new net: IC102.3 (D1), U_ROM9.11 (O0)
- new net: IC102.4 (D2), U_ROM9.12 (O1)
- new net: IC102.7 (D3), U_ROM9.13 (O2)
- new net: IC102.8 (D4), U_ROM9.15 (O3)
- new net: IC102.13 (D5), U_ROM9.16 (O4)
- new net: IC102.14 (D6), U_ROM9.17 (O5)
- new net: IC102.17 (D7), U_ROM9.18 (O6)
- new net: IC102.18 (D8), U_ROM9.19 (O7)
- new net: IC13.13 (I1), IC48.6 (O)
- new net: IC51.12 (O), IC65.1 (I0)
- new net: IC97.13 (D5), U_ROM4.16 (O4)
- new net: IC97.14 (D6), U_ROM4.17 (O5)
- new net: IC97.17 (D7), U_ROM4.18 (O6)
- new net: IC97.18 (D8), U_ROM4.19 (O7)
- new net: IC97.3 (D1), U_ROM4.11 (O0)
- new net: IC97.4 (D2), U_ROM4.12 (O1)
- new net: IC97.7 (D3), U_ROM4.13 (O2)
- new net: IC97.8 (D4), U_ROM4.15 (O3)
- new net: IC80.7 (1Y), IC91.17 (D7)
- new net: IC80.9 (2Y), IC91.18 (D8)
- new net: ALU_HIGH1.7 (CN), ALU_LOW1.16 (CN+4)
- new net: ALU_LOW1.7 (CN), IC_86_1.3 (O)
- new net: IC45.6 (O), IC49.13 (D6)
- new net: IC44.6 (O), IC49.14 (D5)
- new net: IC14.7 (1Y), IC_86_1.1 (I0)
- new net: IC21.4 (O), IC23.13 (I2)
- new net: IC29.3 (O), IC29.4 (I0)
- new net: IC26.12 (4Y), IC40.11 (B4)
- new net: IC26.9 (3Y), IC40.15 (B3)
- new net: IC26.7 (2Y), IC40.2 (B2)
- new net: IC26.4 (1Y), IC40.6 (B1)
- new net: IC40.9 (C4), IC41.7 (C0)
- new net: IC33.7 (1Y), IC47.11 (A1)
- new net: IC33.9 (2Y), IC47.13 (A2)
- new net: IC34.7 (1Y), IC47.15 (A3)
- new net: IC34.9 (2Y), IC47.17 (A4)
- new net: IC13.3 (O), IC17.4 (1C2)
- new net: IC13.8 (O), IC48.5 (I1)
- new net: IC104.3 (D1), U_ROM11.11 (O0)
- new net: IC104.4 (D2), U_ROM11.12 (O1)
- new net: IC104.7 (D3), U_ROM11.13 (O2)
- new net: IC104.8 (D4), U_ROM11.15 (O3)
- new net: IC104.13 (D5), U_ROM11.16 (O4)
- new net: IC104.14 (D6), U_ROM11.17 (O5)
- new net: IC104.17 (D7), U_ROM11.18 (O6)
- new net: IC104.18 (D8), U_ROM11.19 (O7)
- new net: IC23.12 (O), IC24.1 (~{A}/B), IC25.1 (~{A}/B), IC26.1 (~{A}/B), IC27.1 (~{A}/B)
- new net: IC24.12 (4Y), IC38.11 (B4)
- new net: IC24.4 (1Y), IC38.6 (B1)
- new net: IC24.7 (2Y), IC38.2 (B2)
- new net: IC24.9 (3Y), IC38.15 (B3)
- new net: IC1.9 (4Q), IC4.12 (2C2)
- new net: IC2.9 (4Q), IC4.13 (2C3)
- new net: IC2.6 (3Q), IC4.3 (1C3)
- new net: IC1.6 (3Q), IC4.4 (1C2)
- new net: IC28.5 (Y), IC31.4 (1C2), IC34.11 (2C1)
- new net: IC2.2 (1Q), IC3.3 (1C3)
- new net: IC2.5 (2Q), IC3.13 (2C3)
- new net: IC107.13 (D5), U_ROM14.16 (O4)
- new net: IC107.14 (D6), U_ROM14.17 (O5)
- new net: IC107.17 (D7), U_ROM14.18 (O6)
- new net: IC107.18 (D8), U_ROM14.19 (O7)
- new net: IC107.3 (D1), U_ROM14.11 (O0)
- new net: IC107.4 (D2), U_ROM14.12 (O1)
- new net: IC107.7 (D3), U_ROM14.13 (O2)
- new net: IC107.8 (D4), U_ROM14.15 (O3)
- new net: IC1.5 (2Q), IC3.12 (2C2)
- new net: IC1.2 (1Q), IC3.4 (1C2)
- new net: IC94.3 (D1), U_ROM1.11 (O0)
- new net: IC94.4 (D2), U_ROM1.12 (O1)
- new net: IC94.7 (D3), U_ROM1.13 (O2)
- new net: IC94.8 (D4), U_ROM1.15 (O3)
- new net: IC94.13 (D5), U_ROM1.16 (O4)
- new net: IC94.14 (D6), U_ROM1.17 (O5)
- new net: IC94.17 (D7), U_ROM1.18 (O6)
- new net: IC94.18 (D8), U_ROM1.19 (O7)
- new net: IC27.7 (2Y), IC41.2 (B2)
- new net: IC27.4 (1Y), IC41.6 (B1)
- new net GND: ALU_HIGH1.12 (GND), ALU_LOW1.12 (GND), IC10.1 (1G), IC10.15 (2G), IC11.15 (G), IC12.15 (G), IC14.1 (1G), IC14.10 (2C0), IC14.11 (2C1), IC14.12 (2C2), IC14.13 (2C3), IC14.15 (2G), IC14.3 (1C3), IC15.15 (G), IC16.15 (G), IC17.1 (1G), IC17.10 (2C0), IC17.11 (2C1), IC17.12 (2C2), IC17.13 (2C3), IC17.15 (2G), IC17.3 (1C3), IC18.1 (1G), IC18.10 (2C0), IC18.11 (2C1), IC18.12 (2C2), IC18.13 (2C3), IC18.15 (2G), IC19.10 (3B), IC19.11 (3A), IC19.13 (4B), IC19.14 (4A), IC19.15 (G), IC19.5 (2A), IC19.6 (2B), IC20.10 (3B), IC20.11 (3A), IC20.13 (4B), IC20.14 (4A), IC20.15 (G), IC20.5 (2A), IC20.6 (2B), IC22.13 (D5), IC22.14 (D6), IC22.17 (D7), IC22.18 (D8), IC24.11 (3A), IC24.14 (4A), IC24.15 (G), IC24.5 (2A), IC25.11 (3A), IC25.14 (4A), IC25.15 (G), IC25.2 (1A), IC25.5 (2A), IC26.11 (3A), IC26.14 (4A), IC26.15 (G), IC26.2 (1A), IC26.5 (2A), IC27.10 (3B), IC27.11 (3A), IC27.13 (4B), IC27.14 (4A), IC27.15 (G), IC27.2 (1A), IC27.5 (2A), IC28.4 (D0), IC28.7 (G), IC29.1 (I0), IC3.1 (1G), IC3.15 (2G), IC30.15 (G), IC31.1 (1G), IC31.15 (2G), IC32.1 (1G), IC32.15 (2G), IC33.1 (1G), IC33.15 (2G), IC34.1 (1G), IC34.15 (2G), IC38.7 (C0), IC4.1 (1G), IC4.15 (2G), IC41.11 (B4), IC41.12 (A4), IC41.14 (A3), IC41.15 (B3), IC47.1 (G), IC47.19 (G), IC49.7 (G), IC5.1 (1G), IC5.15 (2G), IC50.12 (D7), IC50.13 (D6), IC50.7 (G), IC51.11 (I2), IC6.1 (1G), IC6.15 (2G), IC66.1 (1G), IC66.10 (2C0), IC66.11 (2C1), IC66.12 (2C2), IC66.13 (2C3), IC66.15 (2G), IC67.12 (D7), IC67.13 (D6), IC67.14 (D5), IC67.7 (G), IC68.1 (1G), IC68.10 (2C0), IC68.11 (2C1), IC68.12 (2C2), IC68.13 (2C3), IC68.15 (2G), IC68.4 (1C2), IC69.12 (D7), IC69.13 (D6), IC69.14 (D5), IC69.7 (G), IC7.1 (1G), IC7.15 (2G), IC76.10 (3B), IC76.11 (3A), IC76.13 (4B), IC76.14 (4A), IC76.15 (G), IC76.5 (2A), IC76.6 (2B), IC77.1 (1G), IC77.11 (2C1), IC77.12 (2C2), IC77.13 (2C3), IC77.15 (2G), IC77.3 (1C3), IC77.4 (1C2), IC77.5 (1C1), IC78.1 (1G), IC78.11 (2C1), IC78.12 (2C2), IC78.13 (2C3), IC78.15 (2G), IC78.3 (1C3), IC78.4 (1C2), IC78.5 (1C1), IC79.1 (1G), IC79.11 (2C1), IC79.12 (2C2), IC79.15 (2G), IC79.3 (1C3), IC79.5 (1C1), IC8.1 (1G), IC8.15 (2G), IC80.1 (1G), IC80.12 (2C2), IC80.13 (2C3), IC80.15 (2G), IC80.3 (1C3), IC80.4 (1C2), IC81.1 (1G), IC81.12 (2C2), IC81.13 (2C3), IC81.15 (2G), IC81.3 (1C3), IC81.4 (1C2), IC82.1 (1G), IC82.12 (2C2), IC82.13 (2C3), IC82.15 (2G), IC82.3 (1C3), IC82.4 (1C2), IC83.1 (1G), IC83.12 (2C2), IC83.13 (2C3), IC83.15 (2G), IC83.3 (1C3), IC83.4 (1C2), IC89.15 (G), IC9.1 (1G), IC9.15 (2G), IC91.10 (GND), IC92.10 (GND), IC92.17 (D7), IC92.18 (D8), U_ROM1.1 (A15), U_ROM1.20 (~{CE}), U_ROM1.22 (~{OE}), U_ROM1.27 (A14), U_ROM10.1 (A15), U_ROM10.20 (~{CE}), U_ROM10.22 (~{OE}), U_ROM10.27 (A14), U_ROM11.1 (A15), U_ROM11.20 (~{CE}), U_ROM11.22 (~{OE}), U_ROM11.27 (A14), U_ROM12.1 (A15), U_ROM12.20 (~{CE}), U_ROM12.22 (~{OE}), U_ROM12.27 (A14), U_ROM13.1 (A15), U_ROM13.20 (~{CE}), U_ROM13.22 (~{OE}), U_ROM13.27 (A14), U_ROM14.1 (A15), U_ROM14.20 (~{CE}), U_ROM14.22 (~{OE}), U_ROM14.27 (A14), U_ROM15.1 (A15), U_ROM15.20 (~{CE}), U_ROM15.22 (~{OE}), U_ROM15.27 (A14), U_ROM2.1 (A15), U_ROM2.20 (~{CE}), U_ROM2.22 (~{OE}), U_ROM2.27 (A14), U_ROM3.1 (A15), U_ROM3.20 (~{CE}), U_ROM3.22 (~{OE}), U_ROM3.27 (A14), U_ROM4.1 (A15), U_ROM4.20 (~{CE}), U_ROM4.22 (~{OE}), U_ROM4.27 (A14), U_ROM5.1 (A15), U_ROM5.20 (~{CE}), U_ROM5.22 (~{OE}), U_ROM5.27 (A14), U_ROM6.1 (A15), U_ROM6.20 (~{CE}), U_ROM6.22 (~{OE}), U_ROM6.27 (A14), U_ROM7.1 (A15), U_ROM7.20 (~{CE}), U_ROM7.22 (~{OE}), U_ROM7.27 (A14), U_ROM8.1 (A15), U_ROM8.20 (~{CE}), U_ROM8.22 (~{OE}), U_ROM8.27 (A14), U_ROM9.1 (A15), U_ROM9.20 (~{CE}), U_ROM9.22 (~{OE}), U_ROM9.27 (A14)
- new net VCC: IC22.1 (CLR), IC24.2 (1A), IC79.13 (2C3), IC79.4 (1C2), IC91.20 (VCC), IC92.20 (VCC)
- new net ah_wrt: IC102.9 (Q4)
- new net al_wrt: IC102.6 (Q3)
- new net alu_a_src_0: IC3.14 (A), IC4.14 (A), IC5.14 (A), IC6.14 (A), IC97.15 (Q6)
- new net alu_a_src_1: IC3.2 (B), IC4.2 (B), IC5.2 (B), IC6.2 (B), IC97.16 (Q7)
- new net alu_a_src_2: IC97.19 (Q8)
- new net alu_a_src_3: IC98.2 (Q1)
- new net alu_a_src_4: IC98.5 (Q2)
- new net alu_a_src_5: IC11.1 (~{A}/B), IC12.1 (~{A}/B), IC98.6 (Q3)
- new net alu_b_src_0: IC10.14 (A), IC101.2 (Q1), IC7.14 (A), IC8.14 (A), IC9.14 (A)
- new net alu_b_src_1: IC10.2 (B), IC101.5 (Q2), IC7.2 (B), IC8.2 (B), IC9.2 (B)
- new net alu_b_src_2: IC101.6 (Q3), IC15.1 (~{A}/B), IC16.1 (~{A}/B)
- new net alu_cf: ALU_HIGH1.16 (CN+4), IC_86_1.5 (I1)
- new net alu_cf_in_invert: IC99.6 (Q3), IC_86_1.2 (I1)
- new net alu_cf_in_src_0: IC14.14 (A), IC99.2 (Q1)
- new net alu_cf_in_src_1: IC14.2 (B), IC99.5 (Q2)
- new net alu_cf_out_invert: IC99.15 (Q6), IC_86_1.4 (I0)
- new net alu_final_cf: IC18.5 (1C1), IC67.3 (D1), IC_86_1.6 (O)
- new net alu_mode: ALU_HIGH1.8 (M), ALU_LOW1.8 (M), IC98.19 (Q8)
- new net alu_of: IC20.3 (1B), IC69.3 (D1), IC_04_1.4 (O)
- new net alu_op_0: ALU_HIGH1.6 (S0), ALU_LOW1.6 (S0), IC98.9 (Q4), IC_10_1.1 (I0)
- new net alu_op_1: ALU_HIGH1.5 (S1), ALU_LOW1.5 (S1), IC98.12 (Q5), IC_02_1.3 (I1)
- new net alu_op_2: ALU_HIGH1.4 (S2), ALU_LOW1.4 (S2), IC98.15 (Q6), IC_02_1.2 (I0)
- new net alu_op_3: ALU_HIGH1.3 (S3), ALU_LOW1.3 (S3), IC98.16 (Q7), IC_10_1.2 (I1)
- new net alu_output_0: ALU_LOW1.9 (F0), IC18.4 (1C2), IC28.1 (D3), IC31.12 (2C2), IC31.6 (1C0), IC67.2 (D2)
- new net alu_output_1: ALU_LOW1.10 (F1), IC31.10 (2C0), IC31.5 (1C1), IC32.4 (1C2)
- new net alu_output_2: ALU_LOW1.11 (F2), IC31.11 (2C1), IC32.12 (2C2), IC32.6 (1C0)
- new net alu_output_3: ALU_LOW1.13 (F3), IC32.10 (2C0), IC32.5 (1C1), IC33.4 (1C2)
- new net alu_output_4: ALU_HIGH1.9 (F0), IC32.11 (2C1), IC33.12 (2C2), IC33.6 (1C0)
- new net alu_output_5: ALU_HIGH1.10 (F1), IC33.10 (2C0), IC33.5 (1C1), IC34.4 (1C2)
- new net alu_output_6: ALU_HIGH1.11 (F2), IC33.11 (2C1), IC34.12 (2C2), IC34.6 (1C0)
- new net alu_output_7: ALU_HIGH1.13 (F3), IC18.3 (1C3), IC28.15 (D4), IC31.13 (2C3), IC31.3 (1C3), IC32.13 (2C3), IC32.3 (1C3), IC33.13 (2C3), IC33.3 (1C3), IC34.10 (2C0), IC34.13 (2C3), IC34.3 (1C3), IC34.5 (1C1), IC67.15 (D4)
- new net alu_zf: IC13.1 (I0), IC17.5 (1C1), IC65.12 (O), IC65.3 (I0), IC66.5 (1C1)
- new net any_interruption: IC13.10 (I1), IC29.6 (O)
- new net bh_wrt: IC102.5 (Q2)
- new net bl_wrt: IC102.2 (Q1)
- new net bph_wrt: IC104.6 (Q3)
- new net bpl_wrt: IC104.5 (Q2)
- new net cf_in_src_0: IC67.11 (A), IC99.16 (Q7)
- new net cf_in_src_1: IC67.10 (B), IC99.19 (Q8)
- new net cf_in_src_2: IC100.2 (Q1), IC67.9 (C)
- new net ch_wrt: IC101.19 (Q8)
- new net cl_wrt: IC101.16 (Q7)
- new net clear_all_irqs: IC105.15 (Q6)
- new net clk: FLAGS1.11 (CLK), IC1.11 (CLK), IC2.11 (CLK), IC22.11 (CLK), IC36.11 (CLK), IC42.11 (CLK), IC91.11 (CLK), IC92.11 (CLK)
- new net cond_flag_src: IC30.1 (~{A}/B), IC95.6 (Q3)
- new net cond_invert: IC37.1 (I0), IC95.5 (Q2)
- new net cond_sel_0: IC49.11 (A), IC50.11 (A), IC95.9 (Q4)
- new net cond_sel_1: IC49.10 (B), IC50.10 (B), IC95.12 (Q5)
- new net cond_sel_2: IC49.9 (C), IC50.9 (C), IC95.15 (Q6)
- new net cond_sel_3: IC76.1 (~{A}/B), IC95.16 (Q7)
- new net condition: IC37.2 (I1), IC76.4 (1Y)
- new net data_bus0: IC42.3 (1D)
- new net data_bus1: IC42.4 (2D)
- new net data_bus2: IC42.7 (3D)
- new net data_bus3: IC42.8 (4D)
- new net data_bus4: IC42.13 (5D)
- new net data_bus5: IC42.14 (6D)
- new net data_bus6: IC42.17 (7D)
- new net data_bus7: IC42.18 (8D)
- new net dh_wrt: IC101.15 (Q6)
- new net dih_wrt: IC103.12 (Q5)
- new net dil_wrt: IC103.9 (Q4)
- new net display_reg_load: IC101.9 (Q4)
- new net dl_wrt: IC101.12 (Q5)
- new net dma_req: IC29.5 (I1), IC49.12 (D7)
- new net escape: IC95.19 (Q8)
- new net ext_input: IC50.1 (D3)
- new net final_condition: IC21.3 (I), IC37.3 (O)
- new net flags_4: FLAGS1.12 (Q5), IC5.6 (1C0), IC89.2 (1A)
- new net flags_5: FLAGS1.15 (Q6), IC5.10 (2C0), IC89.5 (2A)
- new net flags_6: FLAGS1.16 (Q7), IC6.6 (1C0), IC89.11 (3A)
- new net flags_7: FLAGS1.19 (Q8), IC6.10 (2C0), IC89.14 (4A)
- new net flags_cf: FLAGS1.5 (Q2), IC14.5 (1C1), IC28.2 (D2), IC3.10 (2C0), IC30.5 (2A), IC67.4 (D0)
- new net flags_of: FLAGS1.9 (Q4), IC30.14 (4A), IC4.10 (2C0), IC69.4 (D0)
- new net flags_sf: FLAGS1.6 (Q3), IC30.11 (3A), IC4.6 (1C0), IC68.6 (1C0)
- new net flags_zf: FLAGS1.2 (Q1), IC3.6 (1C0), IC30.2 (1A), IC65.5 (I2), IC66.6 (1C0)
- new net force_user_ptb: IC106.5 (Q2), IC29.9 (I0)
- new net gh_wrt: IC106.19 (Q8), IC2.1 (G)
- new net gl_wrt: IC1.1 (G), IC106.16 (Q7)
- new net immy_0: IC107.2 (Q1), IC15.2 (1A)
- new net immy_1: IC107.5 (Q2), IC15.5 (2A)
- new net immy_2: IC107.6 (Q3), IC15.11 (3A)
- new net immy_3: IC107.9 (Q4), IC15.14 (4A)
- new net immy_4: IC107.12 (Q5), IC16.2 (1A)
- new net immy_5: IC107.15 (Q6), IC16.5 (2A)
- new net immy_6: IC107.16 (Q7), IC16.11 (3A)
- new net immy_7: IC107.19 (Q8), IC16.14 (4A)
- new net int_pending: IC29.2 (I1), IC35.3 (O), IC50.2 (D2)
- new net int_request: IC35.1 (I0)
- new net ir0: IC42.2 (1Q), IC80.5 (1C1)
- new net ir1: IC42.5 (2Q), IC80.11 (2C1)
- new net ir2: IC42.6 (3Q), IC81.5 (1C1)
- new net ir3: IC42.9 (4Q), IC81.11 (2C1)
- new net ir4: IC42.12 (5Q), IC82.5 (1C1)
- new net ir5: IC42.15 (6Q), IC82.11 (2C1)
- new net ir6: IC42.16 (7Q), IC83.5 (1C1)
- new net ir7: IC42.19 (8Q), IC83.11 (2C1)
- new net ir_wrt: IC42.1 (G), IC96.16 (Q7)
- new net irq_ack: IC105.12 (Q5)
- new net irq_masks_wrt: IC105.6 (Q3)
- new net irq_vector_wrt: IC105.5 (Q2)
- new net kbus0: IC15.3 (1B), IC7.7 (1Y)
- new net kbus1: IC15.6 (2B), IC7.9 (2Y)
- new net kbus2: IC15.10 (3B), IC8.7 (1Y)
- new net kbus3: IC15.13 (4B), IC8.9 (2Y)
- new net kbus4: IC16.3 (1B), IC9.7 (1Y)
- new net kbus5: IC16.6 (2B), IC9.9 (2Y)
- new net kbus6: IC10.7 (1Y), IC16.10 (3B)
- new net kbus7: IC10.9 (2Y), IC16.13 (4B)
- new net mar_in_src: IC105.9 (Q4)
- new net marh_wrt: IC104.2 (Q1)
- new net marl_wrt: IC103.19 (Q8)
- new net mdr_in_src: IC102.12 (Q5)
- new net mdr_out_en: IC102.16 (Q7)
- new net mdr_out_src: IC102.15 (Q6)
- new net mdr_to_pagetable_buffer_en: IC106.2 (Q1)
- new net mdrh_0: IC7.5 (1C1)
- new net mdrh_1: IC7.11 (2C1)
- new net mdrh_2: IC8.5 (1C1)
- new net mdrh_3: IC8.11 (2C1)
- new net mdrh_4: IC9.5 (1C1)
- new net mdrh_5: IC9.11 (2C1)
- new net mdrh_6: IC10.5 (1C1)
- new net mdrh_7: IC10.11 (2C1)
- new net mdrh_wrt: IC103.2 (Q1)
- new net mdrl_0: IC7.6 (1C0)
- new net mdrl_1: IC7.10 (2C0)
- new net mdrl_2: IC8.6 (1C0)
- new net mdrl_3: IC8.10 (2C0)
- new net mdrl_4: IC9.6 (1C0)
- new net mdrl_5: IC9.10 (2C0)
- new net mdrl_6: IC10.6 (1C0)
- new net mdrl_7: IC10.10 (2C0)
- new net mdrl_wrt: IC102.19 (Q8)
- new net mux_a: IC13.11 (O), IC77.14 (A), IC78.14 (A), IC79.14 (A), IC80.14 (A), IC81.14 (A), IC82.14 (A), IC83.14 (A)
- new net mux_b: IC13.6 (O), IC77.2 (B), IC78.2 (B), IC79.2 (B), IC80.2 (B), IC81.2 (B), IC82.2 (B), IC83.2 (B)
- new net of_in_src_0: IC100.9 (Q4), IC69.11 (A)
- new net of_in_src_1: IC100.12 (Q5), IC69.10 (B)
- new net of_in_src_2: IC100.15 (Q6), IC69.9 (C)
- new net page_table_addr_source: IC29.8 (O)
- new net page_table_we: IC105.19 (Q8)
- new net pch_wrt: IC104.12 (Q5)
- new net pcl_wrt: IC104.9 (Q4)
- new net ptb_wrt: IC105.16 (Q7)
- new net rd: IC100.16 (Q7)
- new net rst: IC100.1 (CLR), IC101.1 (CLR), IC102.1 (CLR), IC103.1 (CLR), IC104.1 (CLR), IC105.1 (CLR), IC106.1 (CLR), IC107.1 (CLR), IC108.1 (CLR), IC94.1 (CLR), IC95.1 (CLR), IC96.1 (CLR), IC97.1 (CLR), IC98.1 (CLR), IC99.1 (CLR)
- new net sf_in_src_0: IC100.5 (Q2), IC68.14 (A)
- new net sf_in_src_1: IC100.6 (Q3), IC68.2 (B)
- new net shift_src_0: IC28.11 (A), IC97.2 (Q1)
- new net shift_src_1: IC28.10 (B), IC97.5 (Q2)
- new net shift_src_2: IC28.9 (C), IC97.6 (Q3)
- new net sih_wrt: IC103.16 (Q7)
- new net sil_wrt: IC103.15 (Q6)
- new net sph_wrt: IC104.16 (Q7)
- new net spl_wrt: IC104.15 (Q6)
- new net status_6: IC36.16 (7Q), IC6.5 (1C1)
- new net status_cpu_mode: IC29.10 (I1), IC36.6 (3Q), IC4.5 (1C1), IC50.4 (D0)
- new net status_dir: IC36.19 (8Q), IC50.15 (D4), IC6.11 (2C1)
- new net status_display_reg_load: IC36.15 (6Q), IC5.11 (2C1), IC50.14 (D5)
- new net status_dma_ack: IC3.5 (1C1), IC36.2 (1Q)
- new net status_halt: IC36.12 (5Q), IC5.5 (1C1)
- new net status_irq_enable: IC3.11 (2C1), IC35.2 (I1), IC36.5 (2Q)
- new net status_paging_en: IC36.9 (4Q), IC4.11 (2C1)
- new net status_wrt: IC36.1 (G), IC96.19 (Q8)
- new net tdrh0: IC7.3 (1C3)
- new net tdrh1: IC7.13 (2C3)
- new net tdrh2: IC8.3 (1C3)
- new net tdrh3: IC8.13 (2C3)
- new net tdrh4: IC9.3 (1C3)
- new net tdrh5: IC9.13 (2C3)
- new net tdrh6: IC10.3 (1C3)
- new net tdrh7: IC10.13 (2C3)
- new net tdrh_wrt: IC103.6 (Q3)
- new net tdrl0: IC7.4 (1C2)
- new net tdrl1: IC7.12 (2C2)
- new net tdrl2: IC8.4 (1C2)
- new net tdrl3: IC8.12 (2C2)
- new net tdrl4: IC9.4 (1C2)
- new net tdrl5: IC9.12 (2C2)
- new net tdrl6: IC10.4 (1C2)
- new net tdrl7: IC10.12 (2C2)
- new net tdrl_wrt: IC103.5 (Q2)
- new net typ_0: IC21.9 (I), IC23.1 (I0), IC48.4 (I0), IC94.2 (Q1)
- new net typ_1: IC13.12 (I0), IC13.4 (I0), IC21.1 (I), IC94.5 (Q2)
- new net u_ad0: IC38.5 (A1), IC91.2 (Q1), U_ROM1.10 (A0), U_ROM10.10 (A0), U_ROM11.10 (A0), U_ROM12.10 (A0), U_ROM13.10 (A0), U_ROM14.10 (A0), U_ROM15.10 (A0), U_ROM2.10 (A0), U_ROM3.10 (A0), U_ROM4.10 (A0), U_ROM5.10 (A0), U_ROM6.10 (A0), U_ROM7.10 (A0), U_ROM8.10 (A0), U_ROM9.10 (A0)
- new net u_ad1: IC38.3 (A2), IC91.5 (Q2), U_ROM1.9 (A1), U_ROM10.9 (A1), U_ROM11.9 (A1), U_ROM12.9 (A1), U_ROM13.9 (A1), U_ROM14.9 (A1), U_ROM15.9 (A1), U_ROM2.9 (A1), U_ROM3.9 (A1), U_ROM4.9 (A1), U_ROM5.9 (A1), U_ROM6.9 (A1), U_ROM7.9 (A1), U_ROM8.9 (A1), U_ROM9.9 (A1)
- new net u_ad10: IC40.14 (A3), IC92.6 (Q3), U_ROM1.21 (A10), U_ROM10.21 (A10), U_ROM11.21 (A10), U_ROM12.21 (A10), U_ROM13.21 (A10), U_ROM14.21 (A10), U_ROM15.21 (A10), U_ROM2.21 (A10), U_ROM3.21 (A10), U_ROM4.21 (A10), U_ROM5.21 (A10), U_ROM6.21 (A10), U_ROM7.21 (A10), U_ROM8.21 (A10), U_ROM9.21 (A10)
- new net u_ad11: IC40.12 (A4), IC92.9 (Q4), U_ROM1.23 (A11), U_ROM10.23 (A11), U_ROM11.23 (A11), U_ROM12.23 (A11), U_ROM13.23 (A11), U_ROM14.23 (A11), U_ROM15.23 (A11), U_ROM2.23 (A11), U_ROM3.23 (A11), U_ROM4.23 (A11), U_ROM5.23 (A11), U_ROM6.23 (A11), U_ROM7.23 (A11), U_ROM8.23 (A11), U_ROM9.23 (A11)
- new net u_ad12: IC41.5 (A1), IC92.12 (Q5), U_ROM1.2 (A12), U_ROM10.2 (A12), U_ROM11.2 (A12), U_ROM12.2 (A12), U_ROM13.2 (A12), U_ROM14.2 (A12), U_ROM15.2 (A12), U_ROM2.2 (A12), U_ROM3.2 (A12), U_ROM4.2 (A12), U_ROM5.2 (A12), U_ROM6.2 (A12), U_ROM7.2 (A12), U_ROM8.2 (A12), U_ROM9.2 (A12)
- new net u_ad13: IC41.3 (A2), IC92.15 (Q6), U_ROM1.26 (A13), U_ROM10.26 (A13), U_ROM11.26 (A13), U_ROM12.26 (A13), U_ROM13.26 (A13), U_ROM14.26 (A13), U_ROM15.26 (A13), U_ROM2.26 (A13), U_ROM3.26 (A13), U_ROM4.26 (A13), U_ROM5.26 (A13), U_ROM6.26 (A13), U_ROM7.26 (A13), U_ROM8.26 (A13), U_ROM9.26 (A13)
- new net u_ad2: IC38.14 (A3), IC91.6 (Q3), U_ROM1.8 (A2), U_ROM10.8 (A2), U_ROM11.8 (A2), U_ROM12.8 (A2), U_ROM13.8 (A2), U_ROM14.8 (A2), U_ROM15.8 (A2), U_ROM2.8 (A2), U_ROM3.8 (A2), U_ROM4.8 (A2), U_ROM5.8 (A2), U_ROM6.8 (A2), U_ROM7.8 (A2), U_ROM8.8 (A2), U_ROM9.8 (A2)
- new net u_ad3: IC38.12 (A4), IC91.9 (Q4), U_ROM1.7 (A3), U_ROM10.7 (A3), U_ROM11.7 (A3), U_ROM12.7 (A3), U_ROM13.7 (A3), U_ROM14.7 (A3), U_ROM15.7 (A3), U_ROM2.7 (A3), U_ROM3.7 (A3), U_ROM4.7 (A3), U_ROM5.7 (A3), U_ROM6.7 (A3), U_ROM7.7 (A3), U_ROM8.7 (A3), U_ROM9.7 (A3)
- new net u_ad4: IC39.5 (A1), IC91.12 (Q5), U_ROM1.6 (A4), U_ROM10.6 (A4), U_ROM11.6 (A4), U_ROM12.6 (A4), U_ROM13.6 (A4), U_ROM14.6 (A4), U_ROM15.6 (A4), U_ROM2.6 (A4), U_ROM3.6 (A4), U_ROM4.6 (A4), U_ROM5.6 (A4), U_ROM6.6 (A4), U_ROM7.6 (A4), U_ROM8.6 (A4), U_ROM9.6 (A4)
- new net u_ad5: IC39.3 (A2), IC91.15 (Q6), U_ROM1.5 (A5), U_ROM10.5 (A5), U_ROM11.5 (A5), U_ROM12.5 (A5), U_ROM13.5 (A5), U_ROM14.5 (A5), U_ROM15.5 (A5), U_ROM2.5 (A5), U_ROM3.5 (A5), U_ROM4.5 (A5), U_ROM5.5 (A5), U_ROM6.5 (A5), U_ROM7.5 (A5), U_ROM8.5 (A5), U_ROM9.5 (A5)
- new net u_ad6: IC39.14 (A3), IC91.16 (Q7), U_ROM1.4 (A6), U_ROM10.4 (A6), U_ROM11.4 (A6), U_ROM12.4 (A6), U_ROM13.4 (A6), U_ROM14.4 (A6), U_ROM15.4 (A6), U_ROM2.4 (A6), U_ROM3.4 (A6), U_ROM4.4 (A6), U_ROM5.4 (A6), U_ROM6.4 (A6), U_ROM7.4 (A6), U_ROM8.4 (A6), U_ROM9.4 (A6)
- new net u_ad7: IC39.12 (A4), IC91.19 (Q8), U_ROM1.3 (A7), U_ROM10.3 (A7), U_ROM11.3 (A7), U_ROM12.3 (A7), U_ROM13.3 (A7), U_ROM14.3 (A7), U_ROM15.3 (A7), U_ROM2.3 (A7), U_ROM3.3 (A7), U_ROM4.3 (A7), U_ROM5.3 (A7), U_ROM6.3 (A7), U_ROM7.3 (A7), U_ROM8.3 (A7), U_ROM9.3 (A7)
- new net u_ad8: IC40.5 (A1), IC92.2 (Q1), U_ROM1.25 (A8), U_ROM10.25 (A8), U_ROM11.25 (A8), U_ROM12.25 (A8), U_ROM13.25 (A8), U_ROM14.25 (A8), U_ROM15.25 (A8), U_ROM2.25 (A8), U_ROM3.25 (A8), U_ROM4.25 (A8), U_ROM5.25 (A8), U_ROM6.25 (A8), U_ROM7.25 (A8), U_ROM8.25 (A8), U_ROM9.25 (A8)
- new net u_ad9: IC40.3 (A2), IC92.5 (Q2), U_ROM1.24 (A9), U_ROM10.24 (A9), U_ROM11.24 (A9), U_ROM12.24 (A9), U_ROM13.24 (A9), U_ROM14.24 (A9), U_ROM15.24 (A9), U_ROM2.24 (A9), U_ROM3.24 (A9), U_ROM4.24 (A9), U_ROM5.24 (A9), U_ROM6.24 (A9), U_ROM7.24 (A9), U_ROM8.24 (A9), U_ROM9.24 (A9)
- new net u_adder0: IC38.4 (S1), IC77.6 (1C0)
- new net u_adder1: IC38.1 (S2), IC77.10 (2C0)
- new net u_adder10: IC40.13 (S3), IC82.6 (1C0)
- new net u_adder11: IC40.10 (S4), IC82.10 (2C0)
- new net u_adder12: IC41.4 (S1), IC83.6 (1C0)
- new net u_adder13: IC41.1 (S2), IC83.10 (2C0)
- new net u_adder2: IC38.13 (S3), IC78.6 (1C0)
- new net u_adder3: IC38.10 (S4), IC78.10 (2C0)
- new net u_adder4: IC39.4 (S1), IC79.6 (1C0)
- new net u_adder5: IC39.1 (S2), IC79.10 (2C0)
- new net u_adder6: IC39.13 (S3), IC80.6 (1C0)
- new net u_adder7: IC39.10 (S4), IC80.10 (2C0)
- new net u_adder8: IC40.4 (S1), IC81.6 (1C0)
- new net u_adder9: IC40.1 (S2), IC81.10 (2C0)
- new net u_cf: IC14.4 (1C2), IC18.6 (1C0), IC22.5 (Q2), IC28.3 (D1), IC30.6 (2B)
- new net u_cf_in_src_0: IC18.14 (A), IC96.6 (Q3)
- new net u_cf_in_src_1: IC18.2 (B), IC96.9 (Q4)
- new net u_of: IC20.2 (1A), IC22.9 (Q4), IC30.13 (4B)
- new net u_of_in_src: IC20.1 (~{A}/B), IC96.15 (Q6)
- new net u_offset_0: IC24.3 (1B), IC94.6 (Q3)
- new net u_offset_1: IC24.6 (2B), IC94.9 (Q4)
- new net u_offset_2: IC24.10 (3B), IC94.12 (Q5)
- new net u_offset_3: IC24.13 (4B), IC94.15 (Q6)
- new net u_offset_4: IC25.3 (1B), IC94.16 (Q7)
- new net u_offset_5: IC25.6 (2B), IC94.19 (Q8)
- new net u_offset_6: IC25.10 (3B), IC25.13 (4B), IC26.10 (3B), IC26.13 (4B), IC26.3 (1B), IC26.6 (2B), IC27.3 (1B), IC27.6 (2B), IC95.2 (Q1)
- new net u_sf: IC19.2 (1A), IC22.6 (Q3), IC30.10 (3B), IC_86_1.9 (I0)
- new net u_sf_in_src: IC19.1 (~{A}/B), IC96.12 (Q5)
- new net u_zf: IC13.2 (I1), IC17.6 (1C0), IC22.2 (Q1), IC30.3 (1B)
- new net u_zf_in_src_0: IC17.14 (A), IC96.2 (Q1)
- new net u_zf_in_src_1: IC17.2 (B), IC96.5 (Q2)
- new net upper_flags_wrt: IC105.2 (Q1), IC89.1 (~{A}/B)
- new net vcc: ALU_HIGH1.24 (VCC), ALU_LOW1.24 (VCC), IC14.6 (1C0), IC28.12 (D7), IC28.13 (D6), IC28.14 (D5), IC65.4 (I1), IC_10_1.4 (I1)
- new net w0: IC11.2 (1A)
- new net w1: IC11.5 (2A)
- new net w2: IC11.11 (3A)
- new net w3: IC11.14 (4A)
- new net w4: IC12.2 (1A)
- new net w5: IC12.5 (2A)
- new net w6: IC12.11 (3A)
- new net w7: IC12.14 (4A)
- new net wait: IC50.3 (D1)
- new net wr: IC100.19 (Q8)
- new net xbus0: ALU_LOW1.2 (A0), IC11.4 (1Y)
- new net xbus1: ALU_LOW1.23 (A1), IC11.7 (2Y)
- new net xbus2: ALU_LOW1.21 (A2), IC11.9 (3Y)
- new net xbus3: ALU_LOW1.19 (A3), IC11.12 (4Y)
- new net xbus4: ALU_HIGH1.2 (A0), IC12.4 (1Y)
- new net xbus5: ALU_HIGH1.23 (A1), IC12.7 (2Y)
- new net xbus6: ALU_HIGH1.21 (A2), IC12.9 (3Y)
- new net xbus7: ALU_HIGH1.19 (A3), IC12.12 (4Y), IC_86_2.2 (I1), IC_86_2.4 (I0)
- new net ybus0: ALU_LOW1.1 (B0), IC15.4 (1Y)
- new net ybus1: ALU_LOW1.22 (B1), IC15.7 (2Y)
- new net ybus2: ALU_LOW1.20 (B2), IC15.9 (3Y)
- new net ybus3: ALU_LOW1.18 (B3), IC15.12 (4Y)
- new net ybus4: ALU_HIGH1.1 (B0), IC16.4 (1Y)
- new net ybus5: ALU_HIGH1.22 (B1), IC16.7 (2Y)
- new net ybus6: ALU_HIGH1.20 (B2), IC16.9 (3Y)
- new net ybus7: ALU_HIGH1.18 (B3), IC16.12 (4Y), IC_86_2.5 (I1)
- new net zbus0: IC1.3 (1D), IC2.3 (1D), IC36.3 (1D), IC47.18 (Y1), IC51.1 (I0), IC66.3 (1C3)
- new net zbus1: IC1.4 (2D), IC2.4 (2D), IC36.4 (2D), IC47.16 (Y2), IC51.2 (I1), IC67.1 (D3)
- new net zbus2: IC1.7 (3D), IC2.7 (3D), IC36.7 (3D), IC47.14 (Y3), IC51.13 (I2), IC68.3 (1C3)
- new net zbus3: IC1.8 (4D), IC2.8 (4D), IC36.8 (4D), IC47.12 (Y4), IC51.3 (I0), IC69.1 (D3)
- new net zbus4: IC1.13 (5D), IC2.13 (5D), IC36.13 (5D), IC47.9 (Y1), IC51.4 (I1), IC89.3 (1B)
- new net zbus5: IC1.14 (6D), IC2.14 (6D), IC36.14 (6D), IC47.7 (Y2), IC51.5 (I2), IC89.6 (2B)
- new net zbus6: IC1.17 (7D), IC2.17 (7D), IC36.17 (7D), IC47.5 (Y3), IC51.9 (I0), IC89.10 (3B)
- new net zbus7: IC1.18 (8D), IC19.3 (1B), IC2.18 (8D), IC36.18 (8D), IC47.3 (Y4), IC51.10 (I1), IC68.5 (1C1), IC69.2 (D2), IC89.13 (4B), IC_86_1.10 (I1), IC_86_2.1 (I0)
- new net zbus_in_src_0: IC31.14 (A), IC32.14 (A), IC33.14 (A), IC34.14 (A), IC97.9 (Q4)
- new net zbus_in_src_1: IC31.2 (B), IC32.2 (B), IC33.2 (B), IC34.2 (B), IC97.12 (Q5)
- new net zf_in_src_0: IC66.14 (A), IC99.9 (Q4)
- new net zf_in_src_1: IC66.2 (B), IC99.12 (Q5)
- new net ~{clk}: IC100.11 (CLK), IC101.11 (CLK), IC102.11 (CLK), IC103.11 (CLK), IC104.11 (CLK), IC105.11 (CLK), IC106.11 (CLK), IC107.11 (CLK), IC108.11 (CLK), IC94.11 (CLK), IC95.11 (CLK), IC96.11 (CLK), IC97.11 (CLK), IC98.11 (CLK), IC99.11 (CLK)
- new net ~{rst}: FLAGS1.1 (CLR), IC91.1 (CLR), IC92.1 (CLR)
- no-connect marks 0 -> 49
Other:
- note added: "0"
- note added: "0 = kernel 1 = user"
- note added: "000 = zf 001 = cf 010 = sf 011 = of 100 = s_l neg: s_ge 101 = s_le neg: s_g 001 = u_l neg: u_ge 110 = u_le neg: u_g"
- note added: "1"
- note added: "2"
- note added: "3"
- note added: "74hc32 at ay20"
- note added: "add mux here to create esc opcode"
- note added: "adder"
- note added: "alu"
- note added: "alu output shifted by one"
- note added: "alu_0 is what the carry flag becomes after a shift right alu_7 is what the cf becomes after a shift-left warning: this is not from the zbus~ this is before the alu's output is shifted~"
- note added: "alu_0 is what the carry flag becomes after a shift right operation. warning: this is not from the zbus~ this is before the alu's output is shifted~"
- note added: "alu_mode removed. of is undefined if alu in logic mode anyway."
- note added: "alu_op == add"
- note added: "alu_op == sub"
- note added: "carry in mux"
- note added: "cf"
- note added: "condition source programmer's flags or u_code flags"
- note added: "dma_ack is also used to tri-state the buses when in dma mode."
- note added: "flags"
- note added: "g_h"
- note added: "g_l"
- note added: "halt: use the halt flag to tri-state all buses. do microcode loop to test for interrupts or dma. if no interrupts or dma then just perform tight loop of zero offset. when int or dma appears, jump +1. next microinstr is pre-fetch type, so that int or dma can be executed. pc will be pointing to after halt. interrupts should always clear the halt flag, so that execution goes normally after the int f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"
- note added: "high"
- note added: "if type = branch, and condition = false, then next = +1"
- note added: "int_pending input to conditional is to be used with halt instruction to check if ints are pending. it is also used with the cpu trace mode so that when coming out of the trace microcode loop, we can jump to the interrupts handler if interrupts are pending. without the int_pending conditional it is impossible to execute interrupts when executing in trace mode."
- note added: "ir"
- note added: "low"
- note added: "lt lte ~lt = gte ~lte + gt"
- note added: "microcode 0 to 63 is reserved for cpu startup. fetch at 0x10 trap at 0x20"
- note added: "microcode sequencing"
- note added: "of"
- note added: "removed trace_mode flag from here. (no longer exists)"
- note added: "rewiring the a1/a27 of the roms will be difficult and could damage the wiring and destroy the board."
- note added: "sf"
- note added: "shl: msb goes into cf. lsb replaced by 0 sla: same as shl rol: lsb becomes msb. rlc: msb goes into cf. lsb becomes cf shr: lsb goes into cf. msb replaced by 0 sra: lsb goes into cf. msb is whatever the previous one was ror: msb becomes lsb rrc: msb becomes cf. lsb goes into cf"
- note added: "status"
- note added: "to calculate of when doing shifts we first save the sign of the original number, then when done shifting we save the value of the result. then we do a xor of both values, and the result is the of. the result of the xor is the msb of the result (zbus7). this is why wehave zbus7 as one of the inputs to of another possibility is to first save the sf into the u-flags register before doing the shifts,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"
- note added: "typ1typ0 00 offset 01 branch 10 pre-fetch 11 post_fetch"
- note added: "u-address"
- note added: "u-address mux"
- note added: "u_flags"
- note added: "unused"
- note added: "unused signals"
- note added: "upper bits are a copy of u_offset6. this means this offset is a signed number from -64 to 63"
- note added: "used for sign extension"
- note added: "zf"
