File: hardware/schematics_whole/kicad/main.kicad_sch (KiCad schematic)
At the start: 301 parts, among them IC1 74377N, IC10 74153N, IC100 74273N, IC101 74273N, IC102 74273N, IC103 74273N, IC104 74273N, IC105 74273N, IC106 74273N, IC107 74273N, IC108 74273N, IC109 7427N, IC11 74257N, IC110 74245N, IC111 74257N, IC112 74257N, IC113 7404N, IC114 74377N, IC115 74244N, IC116 74138N, IC117 74244N, IC118 74244N, IC119 74244N, IC12 74257N, IC120 74244N, IC121 7404N, IC122 7420N, IC123 74151N, IC124 74151N, IC125 74151N, IC126 74151N, IC127 74151N, IC128 74151N, IC129 74151N, IC13 7408N, IC130 74151N, IC131 74151N, IC132 74151N, IC133 74151N, IC134 74151N, IC135 74151N, IC136 74151N, IC137 74151N, IC138 74151N, IC139 74151N, IC14 74153N, IC140 74151N, IC141 74151N, IC142 74151N, IC143 74151N, IC144 74151N, IC145 74151N, IC146 74151N, IC147 74151N, IC148 74151N, IC149 74151N, IC15 74257N, IC150 74151N, IC151 74151N, IC152 74151N, IC153 74151N, IC154 74151N, IC155 74257N, IC156 74257N, IC157 74257N, IC158 74257N, IC159 74257N, IC16 74257N, IC160 74257N, IC161 7408N, IC162 7430N, IC163 7404N, IC164 7474N, IC165 7427N, IC166 74153N, IC167 74153N, IC168 74153N, IC169 74153N, IC17 74153N, IC170 7474N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

Commit message: fixing declaration of types and variables inside libraries
Parts:
- removed C1: C, Capacitor_THT:C_Disc_D7.5mm_W4.4mm_P5.00mm, symbol Device:C
Connections:
- net GND: now also IC155.15 (G), IC156.15 (G)
- no-connect marks 162 -> 169
Other:
- moved on the sheet: IC10A, IC11A, IC12A, IC14A, IC15A, IC16A, IC1A, IC2A, IC3A, IC4A, IC5A, IC6A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
